File: LED Box KiCad/ledbox.kicad_pcb (KiCad board)
At the start: 2 copper layers, 80 x 50 mm, 131 parts, among them CON401 AVR_ISP, J201 Bus, J301 IR LED, J302 Button, J401 Power, J402 Power, J403 Power, J404 Port D, J405 Port B, J406 Port C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

Commit message: Kleine Verbesserungen
Parts:
- moved G*** 0.49 mm to (128.3, 101.3)
Routing:
- net /Bus/RX: track 90.3 -> 89.0 mm
Changed lines of the file:
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@@
     (links 254)
     (no_connects 4)
-    (area 98.061904 65 201.938096 135.000001)
+    (area 109.924999 74.924999 190.075001 125.075001)
     (thickness 1.6)
-    (drawings 24)
+    (drawings 22)
     (tracks 591)
     (zones 0)
@@
   )
   (layers
-    (0 F.Cu signal)
-    (31 B.Cu signal)
+    (0 F.Cu signal hide)
+    (31 B.Cu signal hide)
     (32 B.Adhes user)
     (33 F.Adhes user)
@@
     (zone_45_only no)
     (trace_min 0.2)
-    (segment_width 0.2)
+    (segment_width 0.254)
     (edge_width 0.15)
     (via_size 0.6)
@@
   )
   (module LOGO (layer F.Cu)
-    (at 128.708 101.134)
+    (at 128.27 101.346)
     (fp_text reference G*** (at 0 0) (layer F.SilkS) hide
       (effects (font (thickness 0.3)))
@@
     (effects (font (size 1.5 1.5) (thickness 0.3)))
   )
-  (gr_line (start 170.745 93.895) (end 170.745 101.515) (layer B.SilkS) (width 0.2))
-  (gr_line (start 177.73 101.515) (end 177.73 93.895) (layer B.SilkS) (width 0.2))
-  (gr_line (start 149.79 101.515) (end 177.73 101.515) (layer B.SilkS) (width 0.2))
-  (gr_line (start 149.79 93.895) (end 149.79 101.515) (layer B.SilkS) (width 0.2))
-  (gr_line (start 177.73 93.895) (end 149.79 93.895) (layer B.SilkS) (width 0.2))
-  (gr_text "\nLfdNr\nAddr\nTest" (at 177.095 96.435) (layer B.SilkS)
+  (gr_line (start 177.546 101.6) (end 177.546 93.98) (layer B.SilkS) (width 0.254))
+  (gr_line (start 168.148 101.6) (end 177.546 101.6) (layer B.SilkS) (width 0.254))
+  (gr_line (start 177.546 93.98) (end 170.561 93.98) (layer B.SilkS) (width 0.254))
+  (gr_text "LfdNr\nAddr\nTest" (at 177.038 97.79) (layer B.SilkS)
     (effects (font (size 1.5 1.5) (thickness 0.3)) (justify left mirror))
   )
@@
   (segment (start 134.203427 111.675) (end 135.185 111.675) (width 0.25) (layer F.Cu) (net 3))
   (via (at 135.185 111.675) (size 0.6) (drill 0.4) (layers F.Cu B.Cu) (net 3))
-  (segment (start 163.76 108.5) (end 162.49 108.5) (width 0.25) (layer B.Cu) (net 4))
-  (segment (start 147.25 111.04) (end 142.805 115.485) (width 0.25) (layer B.Cu) (net 4))
-  (segment (start 162.49 108.5) (end 161.855 107.865) (width 0.25) (layer B.Cu) (net 4))
-  (segment (start 161.855 107.865) (end 160.585 107.865) (width 0.25) (layer B.Cu) (net 4))
-  (segment (start 160.585 107.865) (end 157.41 111.04) (width 0.25) (layer B.Cu) (net 4))
-  (segment (start 137.09 112.31) (end 134.55 112.31) (width 0.25) (layer B.Cu) (net 4))
-  (segment (start 157.41 111.04) (end 147.25 111.04) (width 0.25) (layer B.Cu) (net 4))
-  (segment (start 142.805 115.485) (end 140.265 115.485) (width 0.25) (layer B.Cu) (net 4))
-  (segment (start 140.265 115.485) (end 137.09 112.31) (width 0.25) (layer B.Cu) (net 4))
+  (segment (start 134.55 112.31) (end 137.09 112.31) (width 0.25) (layer B.Cu) (net 4))
+  (segment (start 160.929998 107.865) (end 161.855 107.865) (width 0.25) (layer B.Cu) (net 4))
+  (segment (start 137.09 112.31) (end 140.265 115.485) (width 0.25) (layer B.Cu) (net 4))
+  (segment (start 157.754998 111.04) (end 160.929998 107.865) (width 0.25) (layer B.Cu) (net 4))
+  (segment (start 140.265 115.485) (end 142.805 115.485) (width 0.25) (layer B.Cu) (net 4))
+  (segment (start 142.805 115.485) (end 147.25 111.04) (width 0.25) (layer B.Cu) (net 4))
+  (segment (start 147.25 111.04) (end 157.754998 111.04) (width 0.25) (layer B.Cu) (net 4))
+  (segment (start 161.855 107.865) (end 162.49 108.5) (width 0.25) (layer B.Cu) (net 4))
+  (segment (start 162.49 108.5) (end 163.76 108.5) (width 0.25) (layer B.Cu) (net 4))
   (segment (start 163.76 108.5) (end 163.76 102.15) (width 0.25) (layer F.Cu) (net 4))
   (via (at 163.76 108.5) (size 0.6) (drill 0.4) (layers F.Cu B.Cu) (net 4))
@@
   (segment (start 137.582 108.5) (end 141.76614 108.5) (width 0.25) (layer F.Cu) (net 6))
   (segment (start 141.76614 108.5) (end 142.40114 107.865) (width 0.25) (layer F.Cu) (net 6))
+  (segment (start 137.582 106.595) (end 139.023 106.595) (width 0.25) (layer F.Cu) (net 7))
+  (segment (start 139.023 106.595) (end 139.192 106.426) (width 0.25) (layer F.Cu) (net 7))
+  (segment (start 139.192 106.426) (end 146.446 106.426) (width 0.25) (layer F.Cu) (net 7))
+  (segment (start 146.446 106.426) (end 147.885 107.865) (width 0.25) (layer F.Cu) (net 7))
+  (segment (start 147.885 107.865) (end 152.09886 107.865) (width 0.25) (layer F.Cu) (net 7))
   (segment (start 137.582 106.595) (end 136.832 106.595) (width 0.25) (layer F.Cu) (net 7))
   (segment (start 136.832 106.595) (end 136.582 106.845) (width 0.25) (layer F.Cu) (net 7))
@@
   (segment (start 136.582 109.639293) (end 136.210305 110.010988) (width 0.25) (layer F.Cu) (net 7))
   (segment (start 136.210305 110.010988) (end 136.210305 110.499897) (width 0.25) (layer F.Cu) (net 7))
-  (segment (start 138.995 105.96) (end 138.36 106.595) (width 0.25) (layer F.Cu) (net 7))
-  (segment (start 138.36 106.595) (end 137.582 106.595) (width 0.25) (layer F.Cu) (net 7))
-  (segment (start 145.98 105.96) (end 138.995 105.96) (width 0.25) (layer F.Cu) (net 7))
-  (segment (start 147.885 107.865) (end 145.98 105.96) (width 0.25) (layer F.Cu) (net 7))
-  (segment (start 152.09886 107.865) (end 147.885 107.865) (width 0.25) (layer F.Cu) (net 7))
   (segment (start 125.025 88.545) (end 121.3 88.545) (width 0.75) (layer F.Cu) (net 8))
   (segment (start 121.3 88.545) (end 120.58 87.825) (width 0.75) (layer F.Cu) (net 8))
@@
   (segment (start 149.506 94.215) (end 150.095 93.626) (width 0.3) (layer F.Cu) (net 21))
   (segment (start 150.095 93.626) (end 150.095 92.31) (width 0.3) (layer F.Cu) (net 21))
+  (segment (start 156.14 102.87) (end 156.14 105.325) (width 0.25) (layer F.Cu) (net 22))
+  (segment (start 156.14 102.87) (end 157.725 101.285) (width 0.25) (layer F.Cu) (net 22))
+  (segment (start 157.725 101.285) (end 157.725 100.245) (width 0.25) (layer F.Cu) (net 22))
   (segment (start 156.14 105.325) (end 156.775 105.96) (width 0.25) (layer F.Cu) (net 22))
   (segment (start 156.775 105.96) (end 158.045 105.96) (width 0.25) (layer F.Cu) (net 22))
-  (segment (start 156.14 102.13) (end 156.14 105.325) (width 0.25) (layer F.Cu) (net 22))
-  (segment (start 157.725 100.245) (end 157.725 100.545) (width 0.25) (layer F.Cu) (net 22))
-  (segment (start 157.725 100.545) (end 156.14 102.13) (width 0.25) (layer F.Cu) (net 22))
   (segment (start 139.604417 113.89401) (end 140.553427 112.945) (width 0.25) (layer F.Cu) (net 22))
   (segment (start 158.045 107.865) (end 158.045 105.96) (width 0.25) (layer F.Cu) (net 22))
@@
   (segment (start 158.045 109.77) (end 158.045 107.865) (width 0.25) (layer F.Cu) (net 22))
   (segment (start 161.22 108.5) (end 161.22 89.45) (width 0.25) (layer F.Cu) (net 23))
-  (segment (start 154.235 86.91) (end 154.235 83.1) (width 0.25) (layer F.Cu) (net 23))
+  (segment (start 155.505 82.465) (end 155.98 82.465) (width 0.25) (layer F.Cu) (net 23))
   (segment (start 161.22 89.45) (end 160.585 88.815) (width 0.25) (layer F.Cu) (net 23))
-  (segment (start 160.585 88.815) (end 156.14 88.815) (width 0.25) (layer F.Cu) (net 23))
-  (segment (start 154.235 83.1) (end 154.87 82.465) (width 0.25) (layer F.Cu) (net 23))
-  (segment (start 156.14 88.815) (end 154.235 86.91) (width 0.25) (layer F.Cu) (net 23))
-  (segment (start 154.87 82.465) (end 155.98 82.465) (width 0.25) (layer F.Cu) (net 23))
+  (segment (start 160.585 88.815) (end 156.845 88.815) (width 0.25) (layer F.Cu) (net 23))
+  (segment (start 154.879999 83.090001) (end 155.505 82.465) (width 0.25) (layer F.Cu) (net 23))
+  (segment (start 156.845 88.815) (end 154.879999 86.849999) (width 0.25) (layer F.Cu) (net 23))
+  (segment (start 154.879999 86.849999) (end 154.879999 83.090001) (width 0.25) (layer F.Cu) (net 23))
   (segment (start 161.22 111.04) (end 161.22 108.5) (width 0.25) (layer B.Cu) (net 23))
   (via (at 161.22 108.5) (size 0.6) (drill 0.4) (layers F.Cu B.Cu) (net 23))
@@
     )
   )
-  (zone (net 0) (net_name "") (layer B.SilkS) (hatch full 0.508)
+  (zone (net 0) (net_name "") (layer B.SilkS) (hatch edge 0.508)
     (connect_pads (clearance 0.2))
-    (min_thickness 0.254)
+    (min_thickness 0.2)
+    (fill yes (arc_segments 16) (thermal_gap 0.508) (thermal_bridge_width 0.508))
+    (polygon
+      (pts
+        (xy 170.688 93.853) (xy 170.688 101.6) (xy 170.434 101.6) (xy 170.434 99.187) (xy 168.148 99.187)
+        (xy 168.148 101.727) (xy 149.86 101.727) (xy 149.86 93.853)
+      )
+    )
+  )
+  (zone (net 0) (net_name "") (layer B.SilkS) (hatch edge 0.508)
+    (connect_pads (clearance 0.2))
+    (min_thickness 0.2)
     (fill yes (arc_segments 16) (thermal_gap 0.508) (thermal_bridge_width 0.508))
     (polygon
       (pts
-        (xy 170.745 93.895) (xy 170.745 98.975) (xy 170.745 101.515) (xy 168.205 101.515) (xy 149.79 101.515)
-        (xy 149.79 93.895)
+        (xy 168.402 99.441) (xy 168.402 101.219) (xy 170.18 101.219) (xy 170.18 99.441)
       )
     )

Commit message: Kleine Verbesserungen
Parts:
- moved REF** 1.32 mm to (137.8, 102.2)
- moved REF** 0.72 mm to (137.8, 103.5)
- moved REF** 0.57 mm to (138.4, 104.1)
- moved REF** 0.57 mm to (137.2, 104.1)
Routing:
- net /Controller/PWM_B: track 17.7 -> 16.9 mm
- net /Controller/LED_IR: track 18.1 -> 17.6 mm
Changed lines of the file:
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@@
     (thickness 1.6)
     (drawings 22)
-    (tracks 591)
+    (tracks 593)
     (zones 0)
     (modules 131)
@@
   )
   (layers
-    (0 F.Cu signal hide)
+    (0 F.Cu signal)
     (31 B.Cu signal hide)
-    (32 B.Adhes user)
-    (33 F.Adhes user)
-    (34 B.Paste user)
-    (35 F.Paste user)
-    (36 B.SilkS user)
-    (37 F.SilkS user)
-    (38 B.Mask user)
-    (39 F.Mask user)
-    (40 Dwgs.User user)
-    (41 Cmts.User user)
-    (42 Eco1.User user)
-    (43 Eco2.User user)
+    (32 B.Adhes user hide)
+    (33 F.Adhes user hide)
+    (34 B.Paste user hide)
+    (35 F.Paste user hide)
+    (36 B.SilkS user hide)
+    (37 F.SilkS user hide)
+    (38 B.Mask user hide)
+    (39 F.Mask user hide)
+    (40 Dwgs.User user hide)
+    (41 Cmts.User user hide)
+    (42 Eco1.User user hide)
+    (43 Eco2.User user hide)
     (44 Edge.Cuts user)
-    (45 Margin user)
-    (46 B.CrtYd user)
-    (47 F.CrtYd user)
-    (48 B.Fab user)
-    (49 F.Fab user)
+    (45 Margin user hide)
+    (46 B.CrtYd user hide)
+    (47 F.CrtYd user hide)
+    (48 B.Fab user hide)
+    (49 F.Fab user hide)
   )
   (setup
-    (last_trace_width 0.25)
+    (last_trace_width 0.3)
     (user_trace_width 0.3)
     (user_trace_width 0.5)
@@
   )
   (module Vias:VIA-10-05 (layer F.Cu)
-    (at 138.995 104.055)
+    (at 138.43 104.14)
     (fp_text reference REF** (at 0 1.27) (layer F.SilkS) hide
       (effects (font (size 1 1) (thickness 0.15)))
@@
   )
   (module Vias:VIA-10-05 (layer F.Cu)
-    (at 138.995 102.785)
+    (at 137.795 102.235)
     (fp_text reference REF** (at 0 1.27) (layer F.SilkS) hide
       (effects (font (size 1 1) (thickness 0.15)))
@@
   )
   (module Vias:VIA-10-05 (layer F.Cu)
-    (at 137.725 102.785)
+    (at 137.795 103.505)
     (fp_text reference REF** (at 0 1.27) (layer F.SilkS) hide
       (effects (font (size 1 1) (thickness 0.15)))
@@
   )
   (module Vias:VIA-10-05 (layer F.Cu)
-    (at 137.725 104.055)
+    (at 137.16 104.14)
     (fp_text reference REF** (at 0 1.27) (layer F.SilkS) hide
       (effects (font (size 1 1) (thickness 0.15)))
@@
   (gr_line (start 110 75) (end 190 75) (layer Edge.Cuts) (width 0.15))
   (gr_line (start 110 125) (end 110 75) (layer Edge.Cuts) (width 0.15))
+  (segment (start 155.825 100.245) (end 155.363 100.245) (width 0.3) (layer F.Cu) (net 1))
+  (segment (start 155.363 100.245) (end 155.118 100) (width 0.3) (layer F.Cu) (net 1))
+  (segment (start 155.118 100) (end 152.45 100) (width 0.3) (layer F.Cu) (net 1))
+  (segment (start 120.58 116.755) (end 120.58 114.85) (width 0.3) (layer F.Cu) (net 1))
+  (segment (start 120.58 114.85) (end 118.04 114.85) (width 0.3) (layer F.Cu) (net 1))
   (segment (start 142.805 88.815) (end 142.805 79.925) (width 0.75) (layer F.Cu) (net 1))
   (segment (start 142.805 90.72) (end 142.805 88.815) (width 0.75) (layer F.Cu) (net 1))
@@
   (segment (start 112.325 107.23) (end 113.595 105.96) (width 0.3) (layer F.Cu) (net 1))
   (segment (start 113.595 112.945) (end 112.325 111.675) (width 0.3) (layer F.Cu) (net 1))
-  (segment (start 120.58 114.85) (end 118.04 114.85) (width 0.3) (layer F.Cu) (net 1))
   (segment (start 118.04 114.85) (end 116.135 112.945) (width 0.3) (layer F.Cu) (net 1))
   (segment (start 116.135 112.945) (end 113.595 112.945) (width 0.3) (layer F.Cu) (net 1))
-  (segment (start 120.58 116.755) (end 120.58 114.85) (width 0.3) (layer F.Cu) (net 1))
   (segment (start 124.39 116.755) (end 120.58 116.755) (width 0.3) (layer F.Cu) (net 1))
   (segment (start 128.907107 118.714893) (end 126.947214 116.755) (width 0.3) (layer F.Cu) (net 1))
   (segment (start 126.947214 116.755) (end 124.39 116.755) (width 0.3) (layer F.Cu) (net 1))
   (segment (start 152.45 100) (end 152.695 100.245) (width 0.25) (layer F.Cu) (net 1))
-  (segment (start 152.695 100.245) (end 155.825 100.245) (width 0.25) (layer F.Cu) (net 1))
   (segment (start 152.65 100.2) (end 152.45 100) (width 0.5) (layer F.Cu) (net 1))
   (segment (start 147.55 100) (end 152.45 100) (width 0.5) (layer F.Cu) (net 1))
@@
   (segment (start 140.665 102.94) (end 143.045 102.94) (width 0.5) (layer F.Cu) (net 38))
   (segment (start 140.665 101.67) (end 140.665 102.94) (width 0.5) (layer F.Cu) (net 38))
-  (segment (start 132.645 95.8) (end 133.125 95.32) (width 0.25) (layer F.Cu) (net 39))
-  (segment (start 133.125 95.32) (end 135.265 95.32) (width 0.25) (layer F.Cu) (net 39))
-  (segment (start 132.645 108.985202) (end 132.645 95.8) (width 0.25) (layer F.Cu) (net 39))
   (segment (start 134.159695 110.499897) (end 132.645 108.985202) (width 0.25) (layer F.Cu) (net 39))
+  (segment (start 132.645 108.985202) (end 132.645 96.66) (width 0.25) (layer F.Cu) (net 39))
+  (segment (start 132.645 96.66) (end 133.985 95.32) (width 0.25) (layer F.Cu) (net 39))
+  (segment (start 133.985 95.32) (end 135.265 95.32) (width 0.25) (layer F.Cu) (net 39))
+  (segment (start 133.28 107.865) (end 133.28 98.565) (width 0.25) (layer F.Cu) (net 40))
+  (segment (start 133.28 98.565) (end 133.985 97.86) (width 0.25) (layer F.Cu) (net 40))
+  (segment (start 133.985 97.86) (end 135.265 97.86) (width 0.25) (layer F.Cu) (net 40))
   (segment (start 135.265 96.59) (end 135.265 97.86) (width 0.25) (layer F.Cu) (net 40))
-  (segment (start 133.28 107.865) (end 133.28 98.34) (width 0.25) (layer F.Cu) (net 40))
-  (segment (start 133.28 98.34) (end 133.76 97.86) (width 0.25) (layer F.Cu) (net 40))
-  (segment (start 133.76 97.86) (end 135.265 97.86) (width 0.25) (layer F.Cu) (net 40))
   (segment (start 132.645 114.215) (end 132.645 108.5) (width 0.25) (layer B.Cu) (net 40))
   (segment (start 132.645 108.5) (end 133.28 107.865) (width 0.25) (layer B.Cu) (net 40))
@@
   (via (at 133.28 113.58) (size 0.6) (drill 0.4) (layers F.Cu B.Cu) (net 41))
   (segment (start 132.714314 113.58) (end 133.28 113.58) (width 0.25) (layer F.Cu) (net 41))
-  (segment (start 136.455 108.5) (end 136.455 102.15) (width 0.25) (layer B.Cu) (net 42))
+  (segment (start 136.455 108.5) (end 136.455 102.9462) (width 0.25) (layer B.Cu) (net 42))
+  (segment (start 135.265 102.94) (end 136.4488 102.94) (width 0.25) (layer F.Cu) (net 42))
+  (segment (start 136.4488 102.94) (end 136.455 102.9462) (width 0.25) (layer F.Cu) (net 42))
+  (via (at 136.455 102.9462) (size 0.6) (drill 0.4) (layers F.Cu B.Cu) (net 42))
   (segment (start 136.455 108.5) (end 141.535 113.58) (width 0.25) (layer B.Cu) (net 42))
   (segment (start 135.265 102.94) (end 135.265 102.15) (width 0.25) (layer F.Cu) (net 42))
   (segment (start 135.265 102.15) (end 135.265 101.67) (width 0.25) (layer F.Cu) (net 42))
-  (segment (start 135.745 102.15) (end 135.265 102.15) (width 0.25) (layer F.Cu) (net 42))
-  (segment (start 136.455 102.15) (end 135.745 102.15) (width 0.25) (layer F.Cu) (net 42))
-  (via (at 136.455 102.15) (size 0.6) (drill 0.4) (layers F.Cu B.Cu) (net 42))
   (segment (start 141.049798 113.58) (end 141.535 113.58) (width 0.25) (layer F.Cu) (net 42))
   (via (at 141.535 113.58) (size 0.6) (drill 0.4) (layers F.Cu B.Cu) (net 42))

Commit message: Gerber Dateien erstellt
Other:
- net class Default: via_dia 0.6 -> 0.7
Changed lines of the file:
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@@
     (links 254)
     (no_connects 4)
-    (area 109.924999 74.924999 190.075001 125.075001)
+    (area -0.5 -0.5 201.938096 135.000001)
     (thickness 1.6)
     (drawings 22)
@@
     (35 F.Paste user hide)
     (36 B.SilkS user hide)
-    (37 F.SilkS user hide)
+    (37 F.SilkS user)
     (38 B.Mask user hide)
     (39 F.Mask user hide)
@@
   )
   (setup
-    (last_trace_width 0.3)
+    (last_trace_width 0.25)
     (user_trace_width 0.3)
     (user_trace_width 0.5)
@@
     (segment_width 0.254)
     (edge_width 0.15)
-    (via_size 0.6)
+    (via_size 0.7)
     (via_drill 0.4)
     (via_min_size 0.4)
@@
     (mod_text_size 1 1)
     (mod_text_width 0.15)
-    (pad_size 1 1)
-    (pad_drill 0)
+    (pad_size 0.7 0.7)
+    (pad_drill 0.4)
     (pad_to_mask_clearance 0.2)
     (aux_axis_origin 0 0)
     (visible_elements FFFFFF7F)
     (pcbplotparams
-      (layerselection 0x000f8_80000001)
+      (layerselection 0x010f8_80000001)
       (usegerberextensions false)
-      (excludeedgelayer false)
+      (excludeedgelayer true)
       (linewidth 0.100000)
-      (plotframeref true)
+      (plotframeref false)
       (viasonmask false)
       (mode 1)
@@
       (outputformat 4)
       (mirror false)
-      (drillshape 2)
+      (drillshape 0)
       (scaleselection 1)
       (outputdirectory output))
@@
     (clearance 0.2)
     (trace_width 0.25)
-    (via_dia 0.6)
+    (via_dia 0.7)
     (via_drill 0.4)
     (uvia_dia 0.3)
@@
     (descr "CP, Radial series, Radial, pin pitch=2.50mm, , diameter=6.3mm, Electrolytic Capacitor")
     (tags "CP Radial series Radial pin pitch 2.50mm  diameter 6.3mm Electrolytic Capacitor")
-    (fp_text reference C501 (at 1.25 -4.46 180) (layer F.SilkS)
+    (fp_text reference C501 (at 5.7085 -0.466 270) (layer F.SilkS)
       (effects (font (size 1 1) (thickness 0.15)))
     )
@@
     (descr "CP, Radial series, Radial, pin pitch=2.50mm, , diameter=6.3mm, Electrolytic Capacitor")
     (tags "CP Radial series Radial pin pitch 2.50mm  diameter 6.3mm Electrolytic Capacitor")
-    (fp_text reference C504 (at 1.25 -4.46 180) (layer F.SilkS)
+    (fp_text reference C504 (at -3.245 0.296 270) (layer F.SilkS)
       (effects (font (size 1 1) (thickness 0.15)))
     )

Commit message: Kleine Veränderungen
Parts:
- added R311: 82, Resistors_SMD:R_0805, F.Cu at (143.7, 99.7)
- C501: footprint Capacitors_THT:CP_Radial_D6.3mm_P2.50mm -> Capacitors_THT:CP_Radial_D5.0mm_P2.00mm
- D201, D202, D501: footprint Diodes_SMD:D_MiniMELF -> Diodes_SMD:D_SOD-123
- R305: value 42 -> 82
- moved R305 0.70 mm to (143.7, 97.8)
- moved REF** 0.70 mm to (116.8, 86.3)
- moved R306 0.56 mm to (143.7, 101.6)
- moved R307 0.07 mm to (143.7, 95.9)
Routing:
- net Net-(R305-Pad2): track 3.60 -> 5.27 mm
- net Net-(D301-Pad6): track 3.21 -> 4.83 mm
- net Net-(R307-Pad2): track 11.3 -> 12.1 mm
- net /Bus/COMM_A: track 15.8 -> 16.4 mm
- net Net-(D301-Pad2): track 11.6 -> 11.1 mm
Other:
- net class Default: via_dia 0.7 -> 0.6; via_drill 0.4 -> 0.3
