File: LED Box KiCad/Bus.sch (KiCad schematic (older format))
At the start: 16 parts, among them J201 Bus, U201 ST485C

Commit message: Board Layout (SMD) fertiggestellt
Parts:
- removed R204: 10k, Resistors_SMD:R_1206, symbol R
- C201, C202, C203: footprint Capacitors_SMD:C_1206 -> Capacitors_SMD:C_0805
- R201, R203: value DNP/10k -> DNP/1k; footprint Resistors_SMD:R_1206 -> Resistors_SMD:R_0805
- R202: footprint Resistors_SMD:R_1206 -> Resistors_THT:R_Axial_DIN0207_L6.3mm_D2.5mm_P7.62mm_Horizontal
- R204: renamed from R205; footprint Resistors_SMD:R_1206 -> Resistors_SMD:R_0805
- R205: renamed from R206; footprint Resistors_SMD:R_1206 -> Resistors_SMD:R_0805
- R206: renamed from R207; footprint Resistors_SMD:R_1206 -> Resistors_SMD:R_0805
- R207: renamed from R208; footprint Resistors_SMD:R_1206 -> Resistors_SMD:R_0805
- R208: renamed from R209; footprint Resistors_SMD:R_1206 -> Resistors_SMD:R_0805
Connections:
- net ~RX_EN is gone; now on net GND: U201.2 (~RE)
Other:
- note added: "R201 und R203 werden genutzt um einen \ndefinierten Zustand auf der Leitung \nzu schaffen, wenn kein Sender aktiv ist.\nMüssen nur auf einer Einheit im Bus \nvorhanden sein (=> Auswerteeineit?)."
- note removed: "R4 und R6 werden genutzt um einen \ndefinierten Zustand auf der Leitung \nzu schaffen, wenn kein Sender aktiv ist.\nMüssen nur auf einer Einheit im Bus \nvorhanden sein (=> Auswerteeineit?)."
Changed lines of the file:
@@
 $EndComp
 $Comp
-L R R206
+L R R205
 U 1 1 59DCBFA2
 P 7250 4500
-F 0 "R206" V 7330 4500 50  0000 C CNN
+F 0 "R205" V 7330 4500 50  0000 C CNN
 F 1 "100" V 7250 4500 50  0000 C CNN
-F 2 "Resistors_SMD:R_1206" V 7180 4500 50  0001 C CNN
+F 2 "Resistors_SMD:R_0805" V 7180 4500 50  0001 C CNN
 F 3 "" H 7250 4500 50  0001 C CNN
 	1    7250 4500
@@
 F 0 "C202" H 7525 4850 50  0000 L CNN
 F 1 "22p" H 7525 4650 50  0000 L CNN
-F 2 "Capacitors_SMD:C_1206" H 7538 4600 50  0001 C CNN
+F 2 "Capacitors_SMD:C_0805" H 7538 4600 50  0001 C CNN
 F 3 "" H 7500 4750 50  0001 C CNN
 	1    7500 4750
@@
 $EndComp
 $Comp
-L R R207
+L R R206
 U 1 1 59DCBFB0
 P 7800 4750
-F 0 "R207" V 7880 4750 50  0000 C CNN
+F 0 "R206" V 7880 4750 50  0000 C CNN
 F 1 "22k" V 7800 4750 50  0000 C CNN
-F 2 "Resistors_SMD:R_1206" V 7730 4750 50  0001 C CNN
+F 2 "Resistors_SMD:R_0805" V 7730 4750 50  0001 C CNN
 F 3 "" H 7800 4750 50  0001 C CNN
 	1    7800 4750
@@
 $EndComp
 $Comp
-L R R209
+L R R208
 U 1 1 59DCBFC5
 P 8500 5350
-F 0 "R209" V 8580 5350 50  0000 C CNN
+F 0 "R208" V 8580 5350 50  0000 C CNN
 F 1 "2k2" V 8500 5350 50  0000 C CNN
-F 2 "Resistors_SMD:R_1206" V 8430 5350 50  0001 C CNN
+F 2 "Resistors_SMD:R_0805" V 8430 5350 50  0001 C CNN
 F 3 "" H 8500 5350 50  0001 C CNN
 	1    8500 5350
@@
 $EndComp
 $Comp
-L R R208
+L R R207
 U 1 1 59DCBFCC
 P 8500 4850
-F 0 "R208" V 8580 4850 50  0000 C CNN
+F 0 "R207" V 8580 4850 50  0000 C CNN
 F 1 "3k3" V 8500 4850 50  0000 C CNN
-F 2 "Resistors_SMD:R_1206" V 8430 4850 50  0001 C CNN
+F 2 "Resistors_SMD:R_0805" V 8430 4850 50  0001 C CNN
 F 3 "" H 8500 4850 50  0001 C CNN
 	1    8500 4850
@@
 F 0 "C203" H 8825 5450 50  0000 L CNN
 F 1 "470p" H 8825 5250 50  0000 L CNN
-F 2 "Capacitors_SMD:C_1206" H 8838 5200 50  0001 C CNN
+F 2 "Capacitors_SMD:C_0805" H 8838 5200 50  0001 C CNN
 F 3 "" H 8800 5350 50  0001 C CNN
 	1    8800 5350
@@
 Text Label 1500 3700 0    60   ~ 0
 TX
-Text Label 6600 3100 3    60   ~ 0
-~RX_EN
 Text Label 6800 3100 3    60   ~ 0
 TX_EN
-Text Label 1500 3500 0    60   ~ 0
-~RX_EN
 Text Label 1500 3400 0    60   ~ 0
 TX_EN
@@
 F 0 "R202" V 3180 3600 50  0000 C CNN
 F 1 "DNP/150" V 3000 3600 50  0000 C CNN
-F 2 "Resistors_SMD:R_1206" V 3030 3600 50  0001 C CNN
+F 2 "Resistors_THT:R_Axial_DIN0207_L6.3mm_D2.5mm_P7.62mm_Horizontal" V 3030 3600 50  0001 C CNN
 F 3 "" H 3100 3600 50  0001 C CNN
 	1    3100 3600
@@
 $Comp
 L R R204
-U 1 1 59DCC33D
-P 6600 3550
-F 0 "R204" V 6680 3550 50  0000 C CNN
-F 1 "10k" V 6600 3550 50  0000 C CNN
-F 2 "Resistors_SMD:R_1206" V 6530 3550 50  0001 C CNN
-F 3 "" H 6600 3550 50  0001 C CNN
-	1    6600 3550
-	-1   0    0    1
-$EndComp
-$Comp
-L R R205
 U 1 1 59DCC344
 P 6800 3550
-F 0 "R205" V 6880 3550 50  0000 C CNN
+F 0 "R204" V 6880 3550 50  0000 C CNN
 F 1 "10k" V 6800 3550 50  0000 C CNN
-F 2 "Resistors_SMD:R_1206" V 6730 3550 50  0001 C CNN
+F 2 "Resistors_SMD:R_0805" V 6730 3550 50  0001 C CNN
 F 3 "" H 6800 3550 50  0001 C CNN
 	1    6800 3550
@@
 $Comp
 L GND #PWR08
-U 1 1 59DCC34B
-P 6600 3800
-F 0 "#PWR08" H 6600 3550 50  0001 C CNN
-F 1 "GND" H 6600 3650 50  0000 C CNN
-F 2 "" H 6600 3800 50  0001 C CNN
-F 3 "" H 6600 3800 50  0001 C CNN
-	1    6600 3800
-	1    0    0    -1
-$EndComp
-$Comp
-L GND #PWR09
 U 1 1 59DCC351
 P 6800 3800
-F 0 "#PWR09" H 6800 3550 50  0001 C CNN
+F 0 "#PWR08" H 6800 3550 50  0001 C CNN
 F 1 "GND" H 6800 3650 50  0000 C CNN
 F 2 "" H 6800 3800 50  0001 C CNN
@@
 P 3100 3150
 F 0 "R201" V 3180 3150 50  0000 C CNN
-F 1 "DNP/10k" V 3000 3150 50  0000 C CNN
-F 2 "Resistors_SMD:R_1206" V 3030 3150 50  0001 C CNN
+F 1 "DNP/1k" V 3000 3150 50  0000 C CNN
+F 2 "Resistors_SMD:R_0805" V 3030 3150 50  0001 C CNN
 F 3 "" H 3100 3150 50  0001 C CNN
 	1    3100 3150
@@
 P 3100 4050
 F 0 "R203" V 3180 4050 50  0000 C CNN
-F 1 "DNP/10k" V 3000 4050 50  0000 C CNN
-F 2 "Resistors_SMD:R_1206" V 3030 4050 50  0001 C CNN
+F 1 "DNP/1k" V 3000 4050 50  0000 C CNN
+F 2 "Resistors_SMD:R_0805" V 3030 4050 50  0001 C CNN
 F 3 "" H 3100 4050 50  0001 C CNN
 	1    3100 4050
@@
 $EndComp
 $Comp
-L +5V #PWR010
+L +5V #PWR09
 U 1 1 59DCC365
 P 3100 2900
-F 0 "#PWR010" H 3100 2750 50  0001 C CNN
+F 0 "#PWR09" H 3100 2750 50  0001 C CNN
 F 1 "+5V" H 3100 3040 50  0000 C CNN
 F 2 "" H 3100 2900 50  0001 C CNN
@@
 $EndComp
 $Comp
-L GND #PWR011
+L GND #PWR010
 U 1 1 59DCC36B
 P 3100 4300
-F 0 "#PWR011" H 3100 4050 50  0001 C CNN
+F 0 "#PWR010" H 3100 4050 50  0001 C CNN
 F 1 "GND" H 3100 4150 50  0000 C CNN
 F 2 "" H 3100 4300 50  0001 C CNN
@@
 $EndComp
 Text Notes 3800 3600 0    60   ~ 0
-R4 und R6 werden genutzt um einen \ndefinierten Zustand auf der Leitung \nzu schaffen, wenn kein Sender aktiv ist.\nMüssen nur auf einer Einheit im Bus \nvorhanden sein (=> Auswerteeineit?).
+R201 und R203 werden genutzt um einen \ndefinierten Zustand auf der Leitung \nzu schaffen, wenn kein Sender aktiv ist.\nMüssen nur auf einer Einheit im Bus \nvorhanden sein (=> Auswerteeineit?).
 Text Notes 1550 5050 0    60   ~ 0
 Neues Bauteil: ST485C \n- viel geringerer Ruhestrom als SN75176 \nBei diesem Sender ist der high side Treiber \nschwächer als der low side Treiber, daher \nmuss die CD Schaltung umgedreht werden.\n
@@
 	1500 3800 1900 3800
 Wire Wire Line
-	1500 3500 1900 3500
+	1800 3500 1900 3500
 Wire Wire Line
 	1500 3400 1900 3400
@@
 	6800 3800 6800 3700
 Wire Wire Line
-	6600 3800 6600 3700
-Wire Wire Line
 	3100 4300 3100 4200
 Wire Wire Line
@@
 Wire Wire Line
 	6800 3100 6800 3400
-Wire Wire Line
-	6600 3400 6600 3100
 $Comp
 L Conn_02x05_Odd_Even J201
@@
 $EndComp
 $Comp
-L +5V #PWR012
+L +5V #PWR011
 U 1 1 59DCC8DA
 P 8450 3650
-F 0 "#PWR012" H 8450 3500 50  0001 C CNN
+F 0 "#PWR011" H 8450 3500 50  0001 C CNN
 F 1 "+5V" H 8450 3790 50  0000 C CNN
 F 2 "" H 8450 3650 50  0001 C CNN
@@
 $EndComp
 $Comp
-L GND #PWR013
+L GND #PWR012
 U 1 1 59DCC8E0
 P 8450 3350
-F 0 "#PWR013" H 8450 3100 50  0001 C CNN
+F 0 "#PWR012" H 8450 3100 50  0001 C CNN
 F 1 "GND" H 8450 3200 50  0000 C CNN
 F 2 "" H 8450 3350 50  0001 C CNN
@@
 $EndComp
 $Comp
-L GND #PWR014
+L GND #PWR013
 U 1 1 59DCC8E6
 P 7650 3850
-F 0 "#PWR014" H 7650 3600 50  0001 C CNN
+F 0 "#PWR013" H 7650 3600 50  0001 C CNN
 F 1 "GND" H 7650 3700 50  0000 C CNN
 F 2 "" H 7650 3850 50  0001 C CNN
@@
 Spannungsversorgung und Bus \nüber 10 Pol Flachbandkabel, \neinmal rund ums Spielfeld. \nAuswerteeinheit (1x pro Spielfeld) \nspeist Spannungsversorgung ein \nund bildet Schnittstelle zur \nAuswertung und Datenübergabe\nbzw. Einstellung.
 $Comp
-L +5V #PWR015
+L +5V #PWR014
 U 1 1 59DCC8EF
 P 7650 3250
-F 0 "#PWR015" H 7650 3100 50  0001 C CNN
+F 0 "#PWR014" H 7650 3100 50  0001 C CNN
 F 1 "+5V" H 7650 3390 50  0000 C CNN
 F 2 "" H 7650 3250 50  0001 C CNN
@@
 Connection ~ 7650 3750
 $Comp
-L +5V #PWR016
+L +5V #PWR015
 U 1 1 59DBB3D1
 P 6100 3300
-F 0 "#PWR016" H 6100 3150 50  0001 C CNN
+F 0 "#PWR015" H 6100 3150 50  0001 C CNN
 F 1 "+5V" H 6100 3440 50  0000 C CNN
 F 2 "" H 6100 3300 50  0001 C CNN
@@
 $EndComp
 $Comp
-L GND #PWR017
+L GND #PWR016
 U 1 1 59DBB3D7
 P 6100 3800
-F 0 "#PWR017" H 6100 3550 50  0001 C CNN
+F 0 "#PWR016" H 6100 3550 50  0001 C CNN
 F 1 "GND" H 6100 3650 50  0000 C CNN
 F 2 "" H 6100 3800 50  0001 C CNN
@@
 F 0 "C201" H 6125 3650 50  0000 L CNN
 F 1 "10u" H 6125 3450 50  0000 L CNN
-F 2 "Capacitors_SMD:C_1206" H 6138 3400 50  0001 C CNN
+F 2 "Capacitors_SMD:C_0805" H 6138 3400 50  0001 C CNN
 F 3 "" H 6100 3550 50  0001 C CNN
 	1    6100 3550
@@
 Text HLabel 1500 3400 0    60   Input ~ 0
 TX_EN
-Text HLabel 1500 3500 0    60   Input ~ 0
-~RX_EN
 Text HLabel 1500 3700 0    60   Input ~ 0
 TX
 Text HLabel 1500 3800 0    60   Output ~ 0
 RX
+$Comp
+L GND #PWR017
+U 1 1 59E09C7D
+P 1800 3900
+F 0 "#PWR017" H 1800 3650 50  0001 C CNN
+F 1 "GND" H 1800 3750 50  0000 C CNN
+F 2 "" H 1800 3900 50  0001 C CNN
+F 3 "" H 1800 3900 50  0001 C CNN
+	1    1800 3900
+	1    0    0    -1
+$EndComp
+Wire Wire Line
+	1800 3900 1800 3500
 $EndSCHEMATC

Commit message: Kleine Veränderungen
Parts:
- D201, D202: footprint Diodes_SMD:D_MiniMELF -> Diodes_SMD:D_SOD-123
- R201, R203: value DNP/1k -> 1k; Populate (none) -> Prototype
- R202: value DNP/150 -> 150; Populate (none) -> Prototype
- U201: Populate (none) -> Yes
Changed lines of the file:
@@
 F 0 "D201" H 6750 4600 50  0000 C CNN
 F 1 "1N4148" H 6750 4400 50  0000 C CNN
-F 2 "Diodes_SMD:D_MiniMELF" H 6750 4500 50  0001 C CNN
+F 2 "Diodes_SMD:D_SOD-123" H 6750 4500 50  0001 C CNN
 F 3 "" H 6750 4500 50  0001 C CNN
 	1    6750 4500
@@
 F 0 "D202" H 6750 4900 50  0000 C CNN
 F 1 "1N4148" H 6750 4700 50  0000 C CNN
-F 2 "Diodes_SMD:D_MiniMELF" H 6750 4800 50  0001 C CNN
+F 2 "Diodes_SMD:D_SOD-123" H 6750 4800 50  0001 C CNN
 F 3 "" H 6750 4800 50  0001 C CNN
 	1    6750 4800
@@
 F 2 "Housings_SOIC:SOIC-8_3.9x4.9mm_Pitch1.27mm" H 2450 4200 60  0001 L CNN
 F 3 "http://www.st.com/content/ccc/resource/technical/document/datasheet/4b/81/a8/cd/8a/72/47/82/CD00002183.pdf/files/CD00002183.pdf/jcr:content/translations/en.CD00002183.pdf" H 2450 4300 60  0001 L CNN
+F 4 "Yes" H 2400 3600 60  0001 C CNN "Populate"
 	1    2400 3600
 	1    0    0    -1
@@
 P 3100 3600
 F 0 "R202" V 3180 3600 50  0000 C CNN
-F 1 "DNP/150" V 3000 3600 50  0000 C CNN
+F 1 "150" V 3000 3600 50  0000 C CNN
 F 2 "Resistors_THT:R_Axial_DIN0207_L6.3mm_D2.5mm_P7.62mm_Horizontal" V 3030 3600 50  0001 C CNN
 F 3 "" H 3100 3600 50  0001 C CNN
+F 4 "Prototype" V 3100 3600 60  0001 C CNN "Populate"
 	1    3100 3600
 	1    0    0    -1
@@
 P 3100 3150
 F 0 "R201" V 3180 3150 50  0000 C CNN
-F 1 "DNP/1k" V 3000 3150 50  0000 C CNN
+F 1 "1k" V 3000 3150 50  0000 C CNN
 F 2 "Resistors_SMD:R_0805" V 3030 3150 50  0001 C CNN
 F 3 "" H 3100 3150 50  0001 C CNN
+F 4 "Prototype" V 3100 3150 60  0001 C CNN "Populate"
 	1    3100 3150
 	1    0    0    -1
@@
 P 3100 4050
 F 0 "R203" V 3180 4050 50  0000 C CNN
-F 1 "DNP/1k" V 3000 4050 50  0000 C CNN
+F 1 "1k" V 3000 4050 50  0000 C CNN
 F 2 "Resistors_SMD:R_0805" V 3030 4050 50  0001 C CNN
 F 3 "" H 3100 4050 50  0001 C CNN
+F 4 "Prototype" V 3100 4050 60  0001 C CNN "Populate"
 	1    3100 4050
 	1    0    0    -1
