File: LED Box KiCad/Controller.sch (KiCad schematic (older format))
At the start: 23 parts, among them CON401 AVR_ISP, J401 Power, J402 Power, J403 Power, J404 Port D, J405 Port B, J406 Port C, J407 ADC6, J408 ADC7, U401 ATMEGA88-20AU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

Commit message: Board Layout (SMD) fertiggestellt
Parts:
- removed J403: Power, Socket_Strips:Socket_Strip_Straight_2x04, symbol Conn_02x04_Odd_Even
- removed J406: Port C, Socket_Strips:Socket_Strip_Straight_1x04, symbol Conn_01x04
- added J403: Power, Socket_Strips:Socket_Strip_Straight_2x05, symbol Conn_02x05_Odd_Even
- added J406: Port C, Socket_Strips:Socket_Strip_Straight_1x05, symbol Conn_01x05
- C401, C402, C403, C404, C405, C406, C407, C408, C409: footprint Capacitors_SMD:C_1206 -> Capacitors_SMD:C_0805
- R401, R402, R403: footprint Resistors_SMD:R_1206 -> Resistors_SMD:R_0805
- U401: footprint TQFP32 -> Housings_QFP:TQFP-32_7x7mm_Pitch0.8mm
Connections:
- net +5V: now also J403.1 (Pin_1), J403.3 (Pin_3), J403.5 (Pin_5), J403.7 (Pin_7), J403.9 (Pin_9)
- net GND: now also J403.10 (Pin_10), J403.2 (Pin_2), J403.4 (Pin_4), J403.6 (Pin_6), J403.8 (Pin_8)
- net LED1: now also J406.2 (Pin_2)
- net LED2: now also J406.3 (Pin_3)
- net PUSH1: now also J406.4 (Pin_4)
- net PUSH2: now also J406.5 (Pin_5)
- net PWM_G: now also U401.13 ((PCINT1/OC1A)PB1); no longer U401.14 ((PCINT2/OC1B/~SS~)PB2)
- net PWM_R: now also U401.14 ((PCINT2/OC1B/~SS~)PB2); no longer U401.13 ((PCINT1/OC1A)PB1)
- net ~RX_EN renamed PC1
- net PC1: now also J406.1 (Pin_1)
Changed lines of the file:
@@
 F 0 "C408" H 7925 2250 50  0000 L CNN
 F 1 "DNP/22p" H 7925 2050 50  0000 L CNN
-F 2 "Capacitors_SMD:C_1206" H 7938 2000 50  0001 C CNN
+F 2 "Capacitors_SMD:C_0805" H 7938 2000 50  0001 C CNN
 F 3 "" H 7900 2150 50  0001 C CNN
 	1    7900 2150
@@
 F 0 "C409" H 8625 2250 50  0000 L CNN
 F 1 "DNP/22p" H 8625 2050 50  0000 L CNN
-F 2 "Capacitors_SMD:C_1206" H 8638 2000 50  0001 C CNN
+F 2 "Capacitors_SMD:C_0805" H 8638 2000 50  0001 C CNN
 F 3 "" H 8600 2150 50  0001 C CNN
 	1    8600 2150
@@
 F 0 "U401" H 1750 3800 50  0000 L BNN
 F 1 "ATMEGA88-20AU" H 2950 1150 50  0000 L BNN
-F 2 "TQFP32" H 2500 2550 50  0001 C CIN
+F 2 "Housings_QFP:TQFP-32_7x7mm_Pitch0.8mm" H 2500 2550 50  0001 C CIN
 F 3 "http://ww1.microchip.com/downloads/en/DeviceDoc/Atmel-2545-8-bit-AVR-Microcontroller-ATmega48-88-168_Datasheet.pdf" H 2500 2550 50  0001 C CNN
 	1    2500 2550
@@
 F 0 "C402" H 4125 6150 50  0000 L CNN
 F 1 "100n" H 4125 5950 50  0000 L CNN
-F 2 "Capacitors_SMD:C_1206" H 4138 5900 50  0001 C CNN
+F 2 "Capacitors_SMD:C_0805" H 4138 5900 50  0001 C CNN
 F 3 "" H 4100 6050 50  0001 C CNN
 	1    4100 6050
@@
 F 0 "C401" H 1375 2150 50  0000 L CNN
 F 1 "100n" H 1375 1950 50  0000 L CNN
-F 2 "Capacitors_SMD:C_1206" H 1388 1900 50  0001 C CNN
+F 2 "Capacitors_SMD:C_0805" H 1388 1900 50  0001 C CNN
 F 3 "" H 1350 2050 50  0001 C CNN
 	1    1350 2050
@@
 F 0 "C403" H 4425 6150 50  0000 L CNN
 F 1 "100n" H 4425 5950 50  0000 L CNN
-F 2 "Capacitors_SMD:C_1206" H 4438 5900 50  0001 C CNN
+F 2 "Capacitors_SMD:C_0805" H 4438 5900 50  0001 C CNN
 F 3 "" H 4400 6050 50  0001 C CNN
 	1    4400 6050
@@
 F 0 "C404" H 4725 6150 50  0000 L CNN
 F 1 "100n" H 4725 5950 50  0000 L CNN
-F 2 "Capacitors_SMD:C_1206" H 4738 5900 50  0001 C CNN
+F 2 "Capacitors_SMD:C_0805" H 4738 5900 50  0001 C CNN
 F 3 "" H 4700 6050 50  0001 C CNN
 	1    4700 6050
@@
 	3900 2900 3500 2900
 Wire Wire Line
-	3900 2400 3500 2400
-Wire Wire Line
 	3900 2300 3500 2300
 Wire Wire Line
@@
 F 0 "R401" V 4230 1750 50  0000 C CNN
 F 1 "1k" V 4150 1750 50  0000 C CNN
-F 2 "Resistors_SMD:R_1206" V 4080 1750 50  0001 C CNN
+F 2 "Resistors_SMD:R_0805" V 4080 1750 50  0001 C CNN
 F 3 "" H 4150 1750 50  0001 C CNN
 	1    4150 1750
@@
 F 0 "R403" V 4530 1850 50  0000 C CNN
 F 1 "1k" V 4450 1850 50  0000 C CNN
-F 2 "Resistors_SMD:R_1206" V 4380 1850 50  0001 C CNN
+F 2 "Resistors_SMD:R_0805" V 4380 1850 50  0001 C CNN
 F 3 "" H 4450 1850 50  0001 C CNN
 	1    4450 1850
@@
 F 0 "R402" V 4230 1950 50  0000 C CNN
 F 1 "1k" V 4150 1950 50  0000 C CNN
-F 2 "Resistors_SMD:R_1206" V 4080 1950 50  0001 C CNN
+F 2 "Resistors_SMD:R_0805" V 4080 1950 50  0001 C CNN
 F 3 "" H 4150 1950 50  0001 C CNN
 	1    4150 1950
@@
 $EndComp
 Wire Wire Line
-	1400 5200 1400 6800
-Wire Wire Line
-	2100 5300 2100 6900
+	1400 5200 1400 6900
+Wire Wire Line
+	2100 5300 2100 7000
 Wire Wire Line
 	2100 5300 2000 5300
@@
 F 0 "C405" H 5025 6150 50  0000 L CNN
 F 1 "100n" H 5025 5950 50  0000 L CNN
-F 2 "Capacitors_SMD:C_1206" H 5038 5900 50  0001 C CNN
+F 2 "Capacitors_SMD:C_0805" H 5038 5900 50  0001 C CNN
 F 3 "" H 5000 6050 50  0001 C CNN
 	1    5000 6050
@@
 F 0 "C406" H 5325 6150 50  0000 L CNN
 F 1 "100n" H 5325 5950 50  0000 L CNN
-F 2 "Capacitors_SMD:C_1206" H 5338 5900 50  0001 C CNN
+F 2 "Capacitors_SMD:C_0805" H 5338 5900 50  0001 C CNN
 F 3 "" H 5300 6050 50  0001 C CNN
 	1    5300 6050
@@
 F 0 "C407" H 5625 6150 50  0000 L CNN
 F 1 "100n" H 5625 5950 50  0000 L CNN
-F 2 "Capacitors_SMD:C_1206" H 5638 5900 50  0001 C CNN
+F 2 "Capacitors_SMD:C_0805" H 5638 5900 50  0001 C CNN
 F 3 "" H 5600 6050 50  0001 C CNN
 	1    5600 6050
@@
 	5000 6200 5000 6300
 Connection ~ 5000 6300
+Text HLabel 3900 1650 2    60   Output ~ 0
+PWM_R
 Text HLabel 3900 1550 2    60   Output ~ 0
-PWM_R
-Text HLabel 3900 1650 2    60   Output ~ 0
 PWM_G
 Text HLabel 3900 2300 2    60   Output ~ 0
 TX_EN
-Text HLabel 3900 2400 2    60   Output ~ 0
-~RX_EN
 Text HLabel 3900 3050 2    60   Input ~ 0
 RX
@@
 Text Label 3900 2800 2    60   ~ 0
 PC5
-Text Label 2900 6500 2    60   ~ 0
+Text Label 2900 6600 2    60   ~ 0
 PC2
-Text Label 2900 6600 2    60   ~ 0
+Text Label 2900 6700 2    60   ~ 0
 PC3
-Text Label 2900 6700 2    60   ~ 0
+Text Label 2900 6800 2    60   ~ 0
 PC4
-Text Label 2900 6800 2    60   ~ 0
+Text Label 2900 6900 2    60   ~ 0
 PC5
-$Comp
-L Conn_01x04 J406
-U 1 1 59DCFC29
-P 2350 6600
-F 0 "J406" H 2350 6800 50  0000 C CNN
-F 1 "Port C" H 2350 6300 50  0000 C CNN
-F 2 "Socket_Strips:Socket_Strip_Straight_1x04" H 2350 6600 50  0001 C CNN
-F 3 "" H 2350 6600 50  0001 C CNN
-	1    2350 6600
-	-1   0    0    -1
-$EndComp
-Wire Wire Line
-	2550 6500 2900 6500
-Wire Wire Line
-	2900 6600 2550 6600
-Wire Wire Line
-	2550 6700 2900 6700
-Wire Wire Line
-	2900 6800 2550 6800
-$Comp
-L Conn_02x04_Odd_Even J403
-U 1 1 59DD01F4
-P 1700 6600
-F 0 "J403" H 1750 6800 50  0000 C CNN
-F 1 "Power" H 1750 6300 50  0000 C CNN
-F 2 "Socket_Strips:Socket_Strip_Straight_2x04" H 1700 6600 50  0001 C CNN
-F 3 "" H 1700 6600 50  0001 C CNN
-	1    1700 6600
-	1    0    0    -1
-$EndComp
+Wire Wire Line
+	2550 6600 2900 6600
+Wire Wire Line
+	2900 6700 2550 6700
+Wire Wire Line
+	2550 6800 2900 6800
+Wire Wire Line
+	2900 6900 2550 6900
 Wire Wire Line
 	2100 6500 2000 6500
@@
 L GND #PWR049
 U 1 1 59DD0A3B
-P 2100 6900
-F 0 "#PWR049" H 2100 6650 50  0001 C CNN
-F 1 "GND" H 2100 6750 50  0000 C CNN
-F 2 "" H 2100 6900 50  0001 C CNN
-F 3 "" H 2100 6900 50  0001 C CNN
-	1    2100 6900
+P 2100 7000
+F 0 "#PWR049" H 2100 6750 50  0001 C CNN
+F 1 "GND" H 2100 6850 50  0000 C CNN
+F 2 "" H 2100 7000 50  0001 C CNN
+F 3 "" H 2100 7000 50  0001 C CNN
+	1    2100 7000
 	1    0    0    -1
 $EndComp
@@
 Text HLabel 3900 2900 2    60   Input ~ 0
 ~RESET
+Text Label 3900 2400 2    60   ~ 0
+PC1
+Wire Wire Line
+	3900 2400 3500 2400
+$Comp
+L Conn_02x05_Odd_Even J403
+U 1 1 59E0B53D
+P 1700 6700
+F 0 "J403" H 1750 7000 50  0000 C CNN
+F 1 "Power" H 1750 6400 50  0000 C CNN
+F 2 "Socket_Strips:Socket_Strip_Straight_2x05" H 1700 6700 50  0001 C CNN
+F 3 "" H 1700 6700 50  0001 C CNN
+	1    1700 6700
+	1    0    0    -1
+$EndComp
+Wire Wire Line
+	2000 6900 2100 6900
+Connection ~ 2100 6900
+Wire Wire Line
+	1400 6900 1500 6900
+Connection ~ 1400 6800
+$Comp
+L Conn_01x05 J406
+U 1 1 59E0BA39
+P 2350 6700
+F 0 "J406" H 2350 7000 50  0000 C CNN
+F 1 "Port C" H 2350 6400 50  0000 C CNN
+F 2 "Socket_Strips:Socket_Strip_Straight_1x05" H 2350 6700 50  0001 C CNN
+F 3 "" H 2350 6700 50  0001 C CNN
+	1    2350 6700
+	-1   0    0    -1
+$EndComp
+Text Label 2900 6500 2    60   ~ 0
+PC1
+Wire Wire Line
+	2550 6500 2900 6500
 $EndSCHEMATC

Commit message: Kleine Veränderungen
Parts:
- removed C406: 100n, Capacitors_SMD:C_0805, symbol C
- C408, C409: value DNP/22p -> 22p; Populate (none) -> Prototype
- Y401: value DNP/20MHz -> 20MHz; Populate (none) -> Prototype
Other:
- moved on the sheet: C407
Changed lines of the file:
@@
 P 8250 1800
 F 0 "Y401" H 8250 1950 50  0000 C CNN
-F 1 "DNP/20MHz" H 8250 1650 50  0000 C CNN
+F 1 "20MHz" H 8250 1650 50  0000 C CNN
 F 2 "Crystals:Crystal_HC49-SD_SMD" H 8250 1800 50  0001 C CNN
 F 3 "" H 8250 1800 50  0001 C CNN
+F 4 "Prototype" H 8250 1800 60  0001 C CNN "Populate"
 	1    8250 1800
 	1    0    0    -1
@@
 P 7900 2150
 F 0 "C408" H 7925 2250 50  0000 L CNN
-F 1 "DNP/22p" H 7925 2050 50  0000 L CNN
+F 1 "22p" H 7925 2050 50  0000 L CNN
 F 2 "Capacitors_SMD:C_0805" H 7938 2000 50  0001 C CNN
 F 3 "" H 7900 2150 50  0001 C CNN
+F 4 "Prototype" H 7900 2150 60  0001 C CNN "Populate"
 	1    7900 2150
 	1    0    0    -1
@@
 P 8600 2150
 F 0 "C409" H 8625 2250 50  0000 L CNN
-F 1 "DNP/22p" H 8625 2050 50  0000 L CNN
+F 1 "22p" H 8625 2050 50  0000 L CNN
 F 2 "Capacitors_SMD:C_0805" H 8638 2000 50  0001 C CNN
 F 3 "" H 8600 2150 50  0001 C CNN
+F 4 "Prototype" H 8600 2150 60  0001 C CNN "Populate"
 	1    8600 2150
 	1    0    0    -1
@@
 	4700 6300 4700 6200
 Wire Wire Line
-	4100 6300 5600 6300
+	4100 6300 5300 6300
 Connection ~ 4400 5800
 Wire Wire Line
@@
 	4700 5800 4700 5900
 Wire Wire Line
-	4100 5800 5600 5800
+	4100 5800 5300 5800
 Wire Wire Line
 	1100 2050 1100 2250
@@
 $EndComp
 $Comp
-L C C406
-U 1 1 59DC5E0A
+L C C407
+U 1 1 59DC5E5E
 P 5300 6050
-F 0 "C406" H 5325 6150 50  0000 L CNN
+F 0 "C407" H 5325 6150 50  0000 L CNN
 F 1 "100n" H 5325 5950 50  0000 L CNN
 F 2 "Capacitors_SMD:C_0805" H 5338 5900 50  0001 C CNN
@@
 	1    0    0    -1
 $EndComp
-$Comp
-L C C407
-U 1 1 59DC5E5E
-P 5600 6050
-F 0 "C407" H 5625 6150 50  0000 L CNN
-F 1 "100n" H 5625 5950 50  0000 L CNN
-F 2 "Capacitors_SMD:C_0805" H 5638 5900 50  0001 C CNN
-F 3 "" H 5600 6050 50  0001 C CNN
-	1    5600 6050
-	1    0    0    -1
-$EndComp
-Wire Wire Line
-	5600 5800 5600 5900
+Wire Wire Line
+	5300 5800 5300 5900
 Connection ~ 4700 5800
-Wire Wire Line
-	5300 5900 5300 5800
-Connection ~ 5300 5800
 Wire Wire Line
 	5000 5900 5000 5800
 Connection ~ 5000 5800
 Wire Wire Line
-	5600 6300 5600 6200
+	5300 6300 5300 6200
 Connection ~ 4700 6300
 Wire Wire Line
-	5300 6200 5300 6300
-Connection ~ 5300 6300
-Wire Wire Line
 	5000 6200 5000 6300

Commit message: Atmega88 gegen Atmega88A getauscht
Parts:
- removed U401: ATMEGA88-20AU, Housings_QFP:TQFP-32_7x7mm_Pitch0.8mm, symbol ATMEGA88-20AU
- added U401: ATMEGA88A-AU, Housings_QFP:TQFP-32_7x7mm_Pitch0.8mm, symbol ATMEGA88A-AU
Connections:
- net +5V: now also U401.18 (AVCC), U401.4 (VCC), U401.6 (VCC)
- net ADC6: now also U401.19 (ADC6)
- net ADC7: now also U401.22 (ADC7)
- net AIN0: now also U401.10 ((PCINT22/OC0A/AIN0)PD6)
- net AIN1: now also U401.11 ((PCINT23/AIN1)PD7)
- net BTN: now also U401.2 ((PCINT20/XCK/T0)PD4)
- net GND: now also U401.21 (GND), U401.3 (GND), U401.5 (GND)
- net LED1: now also U401.25 ((PCINT10/ADC2)PC2)
- net LED2: now also U401.26 ((PCINT11/ADC3)PC3)
- net LED_IR: now also U401.9 ((PCINT21/OC0B/T1)PD5)
- net MISO: now also U401.16 ((PCINT4/MISO)PB4)
- net MOSI: now also U401.15 ((PCINT3/OC2A/MOSI)PB3)
- net PB0: now also U401.12 ((PCINT0/CLKO/ICP1)PB0)
- net PC1: now also U401.24 ((PCINT9/ADC1)PC1)
- net PD2: now also U401.32 ((PCINT18/INT0)PD2)
- net PUSH1: now also U401.27 ((PCINT12/SDA/ADC4)PC4)
- net PUSH2: now also U401.28 ((PCINT13/SCL/ADC5)PC5)
- net PWM_B: now also U401.1 ((PCINT19/OC2B/INT1)PD3)
- net PWM_G: now also U401.13 ((PCINT1/OC1A)PB1)
- net PWM_R: now also U401.14 ((PCINT2/OC1B/~SS~)PB2)
- net RX: now also U401.30 ((PCINT16/RXD)PD0)
- net SCK: now also U401.17 ((PCINT5/SCK)PB5)
- net TX: now also U401.31 ((PCINT17/TXD)PD1)
- net TX_EN: now also U401.23 ((PCINT8/ADC0)PC0)
- net XTAL1: now also U401.7 ((PCINT6/XTAL1/TOSC1)PB6)
- net XTAL2: now also U401.8 ((PCINT7/XTAL2/TOSC2)PB7)
- net ~RESET: now also U401.29 ((PCINT14/~RESET~)PC6)
- net at C401.2: now also U401.20 (AREF)
Changed lines of the file:
@@
 $EndDescr
 $Comp
-L +5V #PWR035
+L +5V #PWR403
 U 1 1 59DB9D21
 P 1500 1350
-F 0 "#PWR035" H 1500 1200 50  0001 C CNN
+F 0 "#PWR403" H 1500 1200 50  0001 C CNN
 F 1 "+5V" H 1500 1490 50  0000 C CNN
 F 2 "" H 1500 1350 50  0001 C CNN
@@
 $EndComp
 $Comp
-L GND #PWR036
+L GND #PWR404
 U 1 1 59DB9D27
 P 1500 3850
-F 0 "#PWR036" H 1500 3600 50  0001 C CNN
+F 0 "#PWR404" H 1500 3600 50  0001 C CNN
 F 1 "GND" H 1500 3700 50  0000 C CNN
 F 2 "" H 1500 3850 50  0001 C CNN
@@
 SCK
 $Comp
-L +5V #PWR037
+L +5V #PWR414
 U 1 1 59DB9D3F
 P 9100 4600
-F 0 "#PWR037" H 9100 4450 50  0001 C CNN
+F 0 "#PWR414" H 9100 4450 50  0001 C CNN
 F 1 "+5V" H 9100 4740 50  0000 C CNN
 F 2 "" H 9100 4600 50  0001 C CNN
@@
 $EndComp
 $Comp
-L GND #PWR038
+L GND #PWR415
 U 1 1 59DB9D45
 P 9100 5000
-F 0 "#PWR038" H 9100 4750 50  0001 C CNN
+F 0 "#PWR415" H 9100 4750 50  0001 C CNN
 F 1 "GND" H 9100 4850 50  0000 C CNN
 F 2 "" H 9100 5000 50  0001 C CNN
@@
 $EndComp
 $Comp
-L GND #PWR039
+L GND #PWR412
 U 1 1 59DB9D60
 P 7900 2400
-F 0 "#PWR039" H 7900 2150 50  0001 C CNN
+F 0 "#PWR412" H 7900 2150 50  0001 C CNN
 F 1 "GND" H 7900 2250 50  0000 C CNN
 F 2 "" H 7900 2400 50  0001 C CNN
@@
 $EndComp
 $Comp
-L GND #PWR040
+L GND #PWR413
 U 1 1 59DB9D66
 P 8600 2400
-F 0 "#PWR040" H 8600 2150 50  0001 C CNN
+F 0 "#PWR413" H 8600 2150 50  0001 C CNN
 F 1 "GND" H 8600 2250 50  0000 C CNN
 F 2 "" H 8600 2400 50  0001 C CNN
@@
 Analog Comparator \nwird verwendet
 $Comp
-L ATMEGA88-20AU U401
-U 1 1 59DB9D91
-P 2500 2550
-F 0 "U401" H 1750 3800 50  0000 L BNN
-F 1 "ATMEGA88-20AU" H 2950 1150 50  0000 L BNN
-F 2 "Housings_QFP:TQFP-32_7x7mm_Pitch0.8mm" H 2500 2550 50  0001 C CIN
-F 3 "http://ww1.microchip.com/downloads/en/DeviceDoc/Atmel-2545-8-bit-AVR-Microcontroller-ATmega48-88-168_Datasheet.pdf" H 2500 2550 50  0001 C CNN
-	1    2500 2550
-	1    0    0    -1
-$EndComp
-$Comp
-L +5V #PWR041
+L +5V #PWR410
 U 1 1 59DBC11C
 P 4100 5700
-F 0 "#PWR041" H 4100 5550 50  0001 C CNN
+F 0 "#PWR410" H 4100 5550 50  0001 C CNN
 F 1 "+5V" H 4100 5840 50  0000 C CNN
 F 2 "" H 4100 5700 50  0001 C CNN
@@
 $EndComp
 $Comp
-L GND #PWR042
+L GND #PWR411
 U 1 1 59DBC122
 P 4100 6400
-F 0 "#PWR042" H 4100 6150 50  0001 C CNN
+F 0 "#PWR411" H 4100 6150 50  0001 C CNN
 F 1 "GND" H 4100 6250 50  0000 C CNN
 F 2 "" H 4100 6400 50  0001 C CNN
@@
 $EndComp
 $Comp
-L GND #PWR043
+L GND #PWR401
 U 1 1 59DBCAA6
 P 1100 2250
-F 0 "#PWR043" H 1100 2000 50  0001 C CNN
+F 0 "#PWR401" H 1100 2000 50  0001 C CNN
 F 1 "GND" H 1100 2100 50  0000 C CNN
 F 2 "" H 1100 2250 50  0001 C CNN
@@
 $EndComp
 $Comp
-L +5V #PWR044
+L +5V #PWR408
 U 1 1 59DC0F73
 P 3750 6250
-F 0 "#PWR044" H 3750 6100 50  0001 C CNN
+F 0 "#PWR408" H 3750 6100 50  0001 C CNN
 F 1 "+5V" H 3750 6390 50  0000 C CNN
 F 2 "" H 3750 6250 50  0001 C CNN
@@
 $EndComp
 $Comp
-L GND #PWR045
+L GND #PWR409
 U 1 1 59DC100E
 P 3750 6650
-F 0 "#PWR045" H 3750 6400 50  0001 C CNN
+F 0 "#PWR409" H 3750 6400 50  0001 C CNN
 F 1 "GND" H 3750 6500 50  0000 C CNN
 F 2 "" H 3750 6650 50  0001 C CNN
@@
 	3750 5650 3450 5650
 $Comp
-L GND #PWR046
+L GND #PWR407
 U 1 1 59DC147E
 P 3750 5850
-F 0 "#PWR046" H 3750 5600 50  0001 C CNN
+F 0 "#PWR407" H 3750 5600 50  0001 C CNN
 F 1 "GND" H 3750 5700 50  0000 C CNN
 F 2 "" H 3750 5850 50  0001 C CNN
@@
 $EndComp
 $Comp
-L +5V #PWR047
+L +5V #PWR406
 U 1 1 59DC14BC
 P 3750 5450
-F 0 "#PWR047" H 3750 5300 50  0001 C CNN
+F 0 "#PWR406" H 3750 5300 50  0001 C CNN
 F 1 "+5V" H 3750 5590 50  0000 C CNN
 F 2 "" H 3750 5450 50  0001 C CNN
@@
 $EndComp
 $Comp
-L +5V #PWR048
+L +5V #PWR402
 U 1 1 59DC2648
 P 1400 5200
-F 0 "#PWR048" H 1400 5050 50  0001 C CNN
+F 0 "#PWR402" H 1400 5050 50  0001 C CNN
 F 1 "+5V" H 1400 5340 50  0000 C CNN
 F 2 "" H 1400 5200 50  0001 C CNN
@@
 Connection ~ 1400 6700
 $Comp
-L GND #PWR049
+L GND #PWR405
 U 1 1 59DD0A3B
 P 2100 7000
-F 0 "#PWR049" H 2100 6750 50  0001 C CNN
+F 0 "#PWR405" H 2100 6750 50  0001 C CNN
 F 1 "GND" H 2100 6850 50  0000 C CNN
 F 2 "" H 2100 7000 50  0001 C CNN
@@
 Wire Wire Line
 	2550 6500 2900 6500
+$Comp
+L ATMEGA88A-AU U401
+U 1 1 59E5004A
+P 2500 2550
+F 0 "U401" H 1750 3800 50  0000 L BNN
+F 1 "ATMEGA88A-AU" H 2900 1150 50  0000 L BNN
+F 2 "Housings_QFP:TQFP-32_7x7mm_Pitch0.8mm" H 2500 2550 50  0001 C CIN
+F 3 "" H 2500 2550 50  0001 C CNN
+	1    2500 2550
+	1    0    0    -1
+$EndComp
 $EndSCHEMATC
