File: LED Box KiCad/Interface.sch (KiCad schematic (older format))
At the start: 21 parts, among them J301 IR LED, J302 Button, SW301 Reset, SW302 Push 1, SW303 Push 2, U301 ULN2003

Commit message: Board Layout (SMD) fertiggestellt
Parts:
- C301, C302: footprint Capacitors_SMD:C_1206 -> Capacitors_SMD:C_0805
- D302, D303: footprint LEDs:LED_1206 -> LEDs:LED_0805
- R301, R302, R303, R304, R305, R306, R307, R308, R309, R310: footprint Resistors_SMD:R_1206 -> Resistors_SMD:R_0805
Connections:
- net +5V: now also D302.2 (A), D303.2 (A), R301.1, R302.1, R303.1, R310.1; no longer J302.1 (Pin_1), R308.1, R309.1, SW301.1, SW302.1, SW303.1
- net BTN: now also J302.1 (Pin_1), R310.2; no longer J302.2 (Pin_2), R310.1
- net GND: now also J302.2 (Pin_2), SW301.2, SW302.2, SW303.2; no longer R301.2, R302.2, R303.2, R310.2
- net LED1: now also R308.2; no longer D302.1 (K)
- net LED2: now also R309.2; no longer D303.1 (K)
- net PUSH1: now also R302.2, SW302.1; no longer R302.1, SW302.2
- net PUSH2: now also R303.2, SW303.1; no longer R303.1, SW303.2
- net ~RESET: now also R301.2, SW301.1; no longer R301.1, SW301.2
- new net: D302.1 (K), R308.1
- new net: D303.1 (K), R309.1
Other:
- moved on the sheet: D302, D303, J302, R301, R302, R303, R308, R309, R310, SW301, SW302, SW303
Changed lines of the file:
@@
 F 0 "R304" V 5330 2700 50  0000 C CNN
 F 1 "150" V 5250 2700 50  0000 C CNN
-F 2 "Resistors_SMD:R_1206" V 5180 2700 50  0001 C CNN
+F 2 "Resistors_SMD:R_0805" V 5180 2700 50  0001 C CNN
 F 3 "" H 5250 2700 50  0001 C CNN
 	1    5250 2700
@@
 F 0 "R305" V 5330 3100 50  0000 C CNN
 F 1 "42" V 5250 3100 50  0000 C CNN
-F 2 "Resistors_SMD:R_1206" V 5180 3100 50  0001 C CNN
+F 2 "Resistors_SMD:R_0805" V 5180 3100 50  0001 C CNN
 F 3 "" H 5250 3100 50  0001 C CNN
 	1    5250 3100
@@
 F 0 "R306" V 5330 3300 50  0000 C CNN
 F 1 "22" V 5250 3300 50  0000 C CNN
-F 2 "Resistors_SMD:R_1206" V 5180 3300 50  0001 C CNN
+F 2 "Resistors_SMD:R_0805" V 5180 3300 50  0001 C CNN
 F 3 "" H 5250 3300 50  0001 C CNN
 	1    5250 3300
@@
 F 0 "R307" V 5330 3500 50  0000 C CNN
 F 1 "22" V 5250 3500 50  0000 C CNN
-F 2 "Resistors_SMD:R_1206" V 5180 3500 50  0001 C CNN
+F 2 "Resistors_SMD:R_0805" V 5180 3500 50  0001 C CNN
 F 3 "" H 5250 3500 50  0001 C CNN
 	1    5250 3500
@@
 L R R310
 U 1 1 59DBA988
-P 7750 4200
-F 0 "R310" V 7830 4200 50  0000 C CNN
-F 1 "10k" V 7750 4200 50  0000 C CNN
-F 2 "Resistors_SMD:R_1206" V 7680 4200 50  0001 C CNN
-F 3 "" H 7750 4200 50  0001 C CNN
-	1    7750 4200
+P 7750 4000
+F 0 "R310" V 7830 4000 50  0000 C CNN
+F 1 "10k" V 7750 4000 50  0000 C CNN
+F 2 "Resistors_SMD:R_0805" V 7680 4000 50  0001 C CNN
+F 3 "" H 7750 4000 50  0001 C CNN
+	1    7750 4000
 	1    0    0    -1
 $EndComp
@@
 L Conn_01x02 J302
 U 1 1 59DBA9A6
-P 8050 3850
-F 0 "J302" H 8050 3950 50  0000 C CNN
-F 1 "Button" H 8050 3650 50  0000 C CNN
-F 2 "Pin_Headers:Pin_Header_Straight_1x02" H 8050 3850 50  0001 C CNN
-F 3 "" H 8050 3850 50  0001 C CNN
-	1    8050 3850
+P 8050 4250
+F 0 "J302" H 8050 4350 50  0000 C CNN
+F 1 "Button" H 8050 4050 50  0000 C CNN
+F 2 "Pin_Headers:Pin_Header_Straight_1x02" H 8050 4250 50  0001 C CNN
+F 3 "" H 8050 4250 50  0001 C CNN
+	1    8050 4250
 	1    0    0    -1
 $EndComp
@@
 $EndComp
 Wire Wire Line
-	7450 3950 7850 3950
+	7450 4250 7850 4250
 Wire Wire Line
 	5950 2700 5400 2700
@@
 	7150 3050 7850 3050
 Wire Wire Line
-	7750 3750 7750 3850
-Wire Wire Line
-	7750 3850 7850 3850
-Wire Wire Line
 	7750 4450 7750 4350
-Wire Wire Line
-	7750 4050 7750 3950
-Connection ~ 7750 3950
 Wire Wire Line
 	7750 3150 7850 3150
@@
 L R R301
 U 1 1 59DBAB66
-P 3500 5450
-F 0 "R301" V 3580 5450 50  0000 C CNN
-F 1 "10k" V 3500 5450 50  0000 C CNN
-F 2 "Resistors_SMD:R_1206" V 3430 5450 50  0001 C CNN
-F 3 "" H 3500 5450 50  0001 C CNN
-	1    3500 5450
-	1    0    0    -1
-$EndComp
-Wire Wire Line
-	3500 5200 3600 5200
-Wire Wire Line
-	3500 5100 3500 5300
+P 3500 4850
+F 0 "R301" V 3580 4850 50  0000 C CNN
+F 1 "10k" V 3500 4850 50  0000 C CNN
+F 2 "Resistors_SMD:R_0805" V 3430 4850 50  0001 C CNN
+F 3 "" H 3500 4850 50  0001 C CNN
+	1    3500 4850
+	1    0    0    -1
+$EndComp
+Wire Wire Line
+	3500 5100 3600 5100
+Wire Wire Line
+	3500 5000 3500 5200
 Wire Wire Line
 	3500 4600 3500 4700
@@
 L SW_Push SW301
 U 1 1 59DBAB71
-P 3500 4900
-F 0 "SW301" H 3550 5000 50  0000 L CNN
-F 1 "Reset" H 3500 4840 50  0000 C CNN
-F 2 "Buttons_Switches_THT:SW_PUSH_6mm_h5mm" H 3500 5100 50  0001 C CNN
-F 3 "" H 3500 5100 50  0001 C CNN
-	1    3500 4900
+P 3500 5400
+F 0 "SW301" H 3550 5500 50  0000 L CNN
+F 1 "Reset" H 3500 5340 50  0000 C CNN
+F 2 "Buttons_Switches_THT:SW_PUSH_6mm_h5mm" H 3500 5600 50  0001 C CNN
+F 3 "" H 3500 5600 50  0001 C CNN
+	1    3500 5400
 	0    1    1    0
 $EndComp
@@
 Wire Wire Line
 	3500 5700 3500 5600
-Connection ~ 3500 5200
+Connection ~ 3500 5100
 $Comp
 L +5V #PWR025
@@
 L R R302
 U 1 1 59DBAB86
-P 4200 5450
-F 0 "R302" V 4280 5450 50  0000 C CNN
-F 1 "10k" V 4200 5450 50  0000 C CNN
-F 2 "Resistors_SMD:R_1206" V 4130 5450 50  0001 C CNN
-F 3 "" H 4200 5450 50  0001 C CNN
-	1    4200 5450
-	1    0    0    -1
-$EndComp
-Wire Wire Line
-	4200 5200 4300 5200
-Wire Wire Line
-	4200 5100 4200 5300
+P 4200 4850
+F 0 "R302" V 4280 4850 50  0000 C CNN
+F 1 "10k" V 4200 4850 50  0000 C CNN
+F 2 "Resistors_SMD:R_0805" V 4130 4850 50  0001 C CNN
+F 3 "" H 4200 4850 50  0001 C CNN
+	1    4200 4850
+	1    0    0    -1
+$EndComp
+Wire Wire Line
+	4200 5100 4300 5100
+Wire Wire Line
+	4200 5000 4200 5200
 Wire Wire Line
 	4200 4600 4200 4700
@@
 L SW_Push SW302
 U 1 1 59DBAB91
-P 4200 4900
-F 0 "SW302" H 4250 5000 50  0000 L CNN
-F 1 "Push 1" H 4200 4840 50  0000 C CNN
-F 2 "Buttons_Switches_THT:SW_PUSH_6mm_h5mm" H 4200 5100 50  0001 C CNN
-F 3 "" H 4200 5100 50  0001 C CNN
-	1    4200 4900
+P 4200 5400
+F 0 "SW302" H 4250 5500 50  0000 L CNN
+F 1 "Push 1" H 4200 5340 50  0000 C CNN
+F 2 "Buttons_Switches_THT:SW_PUSH_6mm_h5mm" H 4200 5600 50  0001 C CNN
+F 3 "" H 4200 5600 50  0001 C CNN
+	1    4200 5400
 	0    1    1    0
 $EndComp
@@
 Wire Wire Line
 	4200 5700 4200 5600
-Connection ~ 4200 5200
+Connection ~ 4200 5100
 $Comp
 L +5V #PWR027
@@
 L R R303
 U 1 1 59DBABA6
-P 4900 5450
-F 0 "R303" V 4980 5450 50  0000 C CNN
-F 1 "10k" V 4900 5450 50  0000 C CNN
-F 2 "Resistors_SMD:R_1206" V 4830 5450 50  0001 C CNN
-F 3 "" H 4900 5450 50  0001 C CNN
-	1    4900 5450
-	1    0    0    -1
-$EndComp
-Wire Wire Line
-	4900 5200 5000 5200
-Wire Wire Line
-	4900 5100 4900 5300
+P 4900 4850
+F 0 "R303" V 4980 4850 50  0000 C CNN
+F 1 "10k" V 4900 4850 50  0000 C CNN
+F 2 "Resistors_SMD:R_0805" V 4830 4850 50  0001 C CNN
+F 3 "" H 4900 4850 50  0001 C CNN
+	1    4900 4850
+	1    0    0    -1
+$EndComp
+Wire Wire Line
+	4900 5100 5000 5100
+Wire Wire Line
+	4900 5000 4900 5200
 Wire Wire Line
 	4900 4600 4900 4700
@@
 L SW_Push SW303
 U 1 1 59DBABB1
-P 4900 4900
-F 0 "SW303" H 4950 5000 50  0000 L CNN
-F 1 "Push 2" H 4900 4840 50  0000 C CNN
-F 2 "Buttons_Switches_THT:SW_PUSH_6mm_h5mm" H 4900 5100 50  0001 C CNN
-F 3 "" H 4900 5100 50  0001 C CNN
-	1    4900 4900
+P 4900 5400
+F 0 "SW303" H 4950 5500 50  0000 L CNN
+F 1 "Push 2" H 4900 5340 50  0000 C CNN
+F 2 "Buttons_Switches_THT:SW_PUSH_6mm_h5mm" H 4900 5600 50  0001 C CNN
+F 3 "" H 4900 5600 50  0001 C CNN
+	1    4900 5400
 	0    1    1    0
 $EndComp
@@
 Wire Wire Line
 	4900 5700 4900 5600
-Connection ~ 4900 5200
+Connection ~ 4900 5100
 $Comp
 L +5V #PWR029
@@
 F 0 "C301" H 6325 3350 50  0000 L CNN
 F 1 "10u" H 6325 3150 50  0000 L CNN
-F 2 "Capacitors_SMD:C_1206" H 6338 3100 50  0001 C CNN
+F 2 "Capacitors_SMD:C_0805" H 6338 3100 50  0001 C CNN
 F 3 "" H 6300 3250 50  0001 C CNN
 	1    6300 3250
@@
 F 0 "C302" H 8425 3200 50  0000 L CNN
 F 1 "100n" H 8425 3000 50  0000 L CNN
-F 2 "Capacitors_SMD:C_1206" H 8438 2950 50  0001 C CNN
+F 2 "Capacitors_SMD:C_0805" H 8438 2950 50  0001 C CNN
 F 3 "" H 8400 3100 50  0001 C CNN
 	1    8400 3100
@@
 Text HLabel 3800 3500 0    60   Input ~ 0
 PWM_B
-Text HLabel 7450 3950 0    60   Output ~ 0
+Text HLabel 7450 4250 0    60   Output ~ 0
 BTN
 $Comp
 L LED D302
 U 1 1 59DCD086
+P 5900 4950
+F 0 "D302" H 5900 5050 50  0000 C CNN
+F 1 "LED1" H 5900 4850 50  0000 C CNN
+F 2 "LEDs:LED_0805" H 5900 4950 50  0001 C CNN
+F 3 "" H 5900 4950 50  0001 C CNN
+	1    5900 4950
+	0    -1   -1   0
+$EndComp
+$Comp
+L R R308
+U 1 1 59DCD11C
 P 5900 5350
-F 0 "D302" H 5900 5450 50  0000 C CNN
-F 1 "LED1" H 5900 5250 50  0000 C CNN
-F 2 "LEDs:LED_1206" H 5900 5350 50  0001 C CNN
+F 0 "R308" V 5980 5350 50  0000 C CNN
+F 1 "430" V 5900 5350 50  0000 C CNN
+F 2 "Resistors_SMD:R_0805" V 5830 5350 50  0001 C CNN
 F 3 "" H 5900 5350 50  0001 C CNN
 	1    5900 5350
-	0    -1   -1   0
-$EndComp
-$Comp
-L R R308
-U 1 1 59DCD11C
-P 5900 4950
-F 0 "R308" V 5980 4950 50  0000 C CNN
-F 1 "430" V 5900 4950 50  0000 C CNN
-F 2 "Resistors_SMD:R_1206" V 5830 4950 50  0001 C CNN
-F 3 "" H 5900 4950 50  0001 C CNN
-	1    5900 4950
 	1    0    0    -1
 $EndComp
@@
 	1    0    0    -1
 $EndComp
-Text HLabel 3600 5200 2    60   Output ~ 0
+Text HLabel 3600 5100 2    60   Output ~ 0
 ~RESET
-Text HLabel 4300 5200 2    60   Output ~ 0
+Text HLabel 4300 5100 2    60   Output ~ 0
 PUSH1
-Text HLabel 5000 5200 2    60   Output ~ 0
+Text HLabel 5000 5100 2    60   Output ~ 0
 PUSH2
 Text HLabel 5800 5600 0    60   Input ~ 0
@@
 L LED D303
 U 1 1 59DCD70E
+P 6600 4950
+F 0 "D303" H 6600 5050 50  0000 C CNN
+F 1 "LED2" H 6600 4850 50  0000 C CNN
+F 2 "LEDs:LED_0805" H 6600 4950 50  0001 C CNN
+F 3 "" H 6600 4950 50  0001 C CNN
+	1    6600 4950
+	0    -1   -1   0
+$EndComp
+$Comp
+L R R309
+U 1 1 59DCD714
 P 6600 5350
-F 0 "D303" H 6600 5450 50  0000 C CNN
-F 1 "LED2" H 6600 5250 50  0000 C CNN
-F 2 "LEDs:LED_1206" H 6600 5350 50  0001 C CNN
+F 0 "R309" V 6680 5350 50  0000 C CNN
+F 1 "430" V 6600 5350 50  0000 C CNN
+F 2 "Resistors_SMD:R_0805" V 6530 5350 50  0001 C CNN
 F 3 "" H 6600 5350 50  0001 C CNN
 	1    6600 5350
-	0    -1   -1   0
-$EndComp
-$Comp
-L R R309
-U 1 1 59DCD714
-P 6600 4950
-F 0 "R309" V 6680 4950 50  0000 C CNN
-F 1 "430" V 6600 4950 50  0000 C CNN
-F 2 "Resistors_SMD:R_1206" V 6530 4950 50  0001 C CNN
-F 3 "" H 6600 4950 50  0001 C CNN
-	1    6600 4950
 	1    0    0    -1
 $EndComp
@@
 Wire Wire Line
 	6600 5600 6600 5500
+Wire Wire Line
+	7750 4350 7850 4350
+Wire Wire Line
+	7750 4250 7750 4150
+Connection ~ 7750 4250
+Wire Wire Line
+	7750 3850 7750 3750
 $EndSCHEMATC

Commit message: Kleine Veränderungen
Parts:
- added R311: 82, Resistors_SMD:R_0805, symbol R
- R305: value 42 -> 82
Connections:
- net at R305.2, U301.14 (O3), U301.15 (O2): now also R311.2
- net at D301.6 (RK), R305.1: now also R311.1
Other:
- note removed: "!rund 110mW!"
- moved on the sheet: C301, D301, R304
Changed lines of the file:
@@
 L R R304
 U 1 1 59DBA966
-P 5250 2700
-F 0 "R304" V 5330 2700 50  0000 C CNN
-F 1 "150" V 5250 2700 50  0000 C CNN
-F 2 "Resistors_SMD:R_0805" V 5180 2700 50  0001 C CNN
-F 3 "" H 5250 2700 50  0001 C CNN
-	1    5250 2700
+P 5350 2700
+F 0 "R304" V 5430 2700 50  0000 C CNN
+F 1 "150" V 5350 2700 50  0000 C CNN
+F 2 "Resistors_SMD:R_0805" V 5280 2700 50  0001 C CNN
+F 3 "" H 5350 2700 50  0001 C CNN
+	1    5350 2700
 	0    1    1    0
 $EndComp
@@
 P 5250 3100
 F 0 "R305" V 5330 3100 50  0000 C CNN
-F 1 "42" V 5250 3100 50  0000 C CNN
+F 1 "82" V 5250 3100 50  0000 C CNN
 F 2 "Resistors_SMD:R_0805" V 5180 3100 50  0001 C CNN
 F 3 "" H 5250 3100 50  0001 C CNN
@@
 L +5V #PWR019
 U 1 1 59DBA982
-P 6000 3000
-F 0 "#PWR019" H 6000 2850 50  0001 C CNN
-F 1 "+5V" H 6000 3140 50  0000 C CNN
-F 2 "" H 6000 3000 50  0001 C CNN
-F 3 "" H 6000 3000 50  0001 C CNN
-	1    6000 3000
+P 6100 3000
+F 0 "#PWR019" H 6100 2850 50  0001 C CNN
+F 1 "+5V" H 6100 3140 50  0000 C CNN
+F 2 "" H 6100 3000 50  0001 C CNN
+F 3 "" H 6100 3000 50  0001 C CNN
+	1    6100 3000
 	1    0    0    -1
 $EndComp
@@
 	1    0    0    -1
 $EndComp
-Text Notes 5550 3050 2    60   ~ 0
-!rund 110mW!
 $Comp
 L LRTBG6TG D301
 U 1 1 59DBA991
-P 5700 3300
-F 0 "D301" H 5700 3670 50  0000 C CNN
-F 1 "LRTBG6TG" H 5700 2950 50  0000 C CNN
-F 2 "ledbox-newfootprints:LED-6-BIG" H 5700 2750 50  0001 C CNN
-F 3 "http://www.osram-os.com/Graphics/XPic4/00067263_0.pdf" H 5700 2850 50  0001 C CNN
-	1    5700 3300
-	1    0    0    -1
-$EndComp
-Text Label 5950 2700 2    60   ~ 0
+P 5800 3300
+F 0 "D301" H 5800 3670 50  0000 C CNN
+F 1 "LRTBG6TG" H 5800 2950 50  0000 C CNN
+F 2 "ledbox-newfootprints:LED-6-BIG" H 5800 2750 50  0001 C CNN
+F 3 "http://www.osram-os.com/Graphics/XPic4/00067263_0.pdf" H 5800 2850 50  0001 C CNN
+	1    5800 3300
+	1    0    0    -1
+$EndComp
+Text Label 6050 2700 2    60   ~ 0
 IR_LED_DRV
 Text Label 7150 3050 0    60   ~ 0
@@
 	7450 4250 7850 4250
 Wire Wire Line
-	5950 2700 5400 2700
-Wire Wire Line
-	6000 3100 5900 3100
-Wire Wire Line
-	5400 3500 5500 3500
-Wire Wire Line
-	5400 3300 5500 3300
-Wire Wire Line
-	5400 3100 5500 3100
-Wire Wire Line
-	5000 2700 5100 2700
+	6050 2700 5500 2700
+Wire Wire Line
+	6100 3100 6000 3100
+Wire Wire Line
+	5400 3500 5600 3500
+Wire Wire Line
+	5400 3300 5600 3300
+Wire Wire Line
+	5400 3100 5600 3100
+Wire Wire Line
+	4900 2700 5200 2700
 Wire Wire Line
 	3900 3200 4000 3200
@@
 	4800 3000 4900 3000
 Wire Wire Line
-	4800 2900 5000 2900
-Wire Wire Line
-	5000 2900 5000 2700
+	4800 2900 4900 2900
+Wire Wire Line
+	4900 2900 4900 2700
 Wire Wire Line
 	7150 3050 7850 3050
@@
 Connection ~ 4900 3500
 Wire Wire Line
-	6000 3000 6000 3500
-Wire Wire Line
-	6000 3300 5900 3300
-Connection ~ 6000 3100
-Wire Wire Line
-	6000 3500 5900 3500
-Connection ~ 6000 3300
+	6100 3000 6100 3500
+Wire Wire Line
+	6100 3300 6000 3300
+Connection ~ 6100 3100
+Wire Wire Line
+	6100 3500 6000 3500
+Connection ~ 6100 3300
 $Comp
 L +5V #PWR023
@@
 L +5V #PWR029
 U 1 1 59DBB492
-P 6300 3000
-F 0 "#PWR029" H 6300 2850 50  0001 C CNN
-F 1 "+5V" H 6300 3140 50  0000 C CNN
-F 2 "" H 6300 3000 50  0001 C CNN
-F 3 "" H 6300 3000 50  0001 C CNN
-	1    6300 3000
+P 6400 3000
+F 0 "#PWR029" H 6400 2850 50  0001 C CNN
+F 1 "+5V" H 6400 3140 50  0000 C CNN
+F 2 "" H 6400 3000 50  0001 C CNN
+F 3 "" H 6400 3000 50  0001 C CNN
+	1    6400 3000
 	1    0    0    -1
 $EndComp
@@
 L GND #PWR030
 U 1 1 59DBB498
-P 6300 3500
-F 0 "#PWR030" H 6300 3250 50  0001 C CNN
-F 1 "GND" H 6300 3350 50  0000 C CNN
-F 2 "" H 6300 3500 50  0001 C CNN
-F 3 "" H 6300 3500 50  0001 C CNN
-	1    6300 3500
+P 6400 3500
+F 0 "#PWR030" H 6400 3250 50  0001 C CNN
+F 1 "GND" H 6400 3350 50  0000 C CNN
+F 2 "" H 6400 3500 50  0001 C CNN
+F 3 "" H 6400 3500 50  0001 C CNN
+	1    6400 3500
 	1    0    0    -1
 $EndComp
@@
 L C C301
 U 1 1 59DBB49E
-P 6300 3250
-F 0 "C301" H 6325 3350 50  0000 L CNN
-F 1 "10u" H 6325 3150 50  0000 L CNN
-F 2 "Capacitors_SMD:C_0805" H 6338 3100 50  0001 C CNN
-F 3 "" H 6300 3250 50  0001 C CNN
-	1    6300 3250
-	1    0    0    -1
-$EndComp
-Wire Wire Line
-	6300 3400 6300 3500
-Wire Wire Line
-	6300 3000 6300 3000
-Wire Wire Line
-	6300 3000 6300 3100
+P 6400 3250
+F 0 "C301" H 6425 3350 50  0000 L CNN
+F 1 "10u" H 6425 3150 50  0000 L CNN
+F 2 "Capacitors_SMD:C_0805" H 6438 3100 50  0001 C CNN
+F 3 "" H 6400 3250 50  0001 C CNN
+	1    6400 3250
+	1    0    0    -1
+$EndComp
+Wire Wire Line
+	6400 3400 6400 3500
+Wire Wire Line
+	6400 3000 6400 3000
+Wire Wire Line
+	6400 3000 6400 3100
 $Comp
 L +5V #PWR031
@@
 Wire Wire Line
 	7750 3850 7750 3750
+$Comp
+L R R311
+U 1 1 59E4B05C
+P 5250 2900
+F 0 "R311" V 5330 2900 50  0000 C CNN
+F 1 "82" V 5250 2900 50  0000 C CNN
+F 2 "Resistors_SMD:R_0805" V 5180 2900 50  0001 C CNN
+F 3 "" H 5250 2900 50  0001 C CNN
+	1    5250 2900
+	0    1    1    0
+$EndComp
+Wire Wire Line
+	5100 2900 5000 2900
+Wire Wire Line
+	5000 2900 5000 3100
+Connection ~ 5000 3100
+Wire Wire Line
+	5400 2900 5500 2900
+Wire Wire Line
+	5500 2900 5500 3100
+Connection ~ 5500 3100
 $EndSCHEMATC
