File: LED Box KiCad/Supply.sch (KiCad schematic (older format))
At the start: 8 parts, among them J501 6.5V-12V, J502 5V, U501 AZ1117-5.0

Commit message: Board Layout (SMD) fertiggestellt
Parts:
- added D502: LED2, LEDs:LED_0805, symbol LED
- added R501: 430, Resistors_SMD:R_0805, symbol R
- C501, C504: footprint Capacitors_SMD:CP_Elec_4x5.7 -> Capacitors_THT:CP_Radial_D6.3mm_P2.50mm
- C502, C503: footprint Capacitors_SMD:C_1206 -> Capacitors_SMD:C_0805
- U501: footprint TO_SOT_Packages_SMD:TO-263-3Lead -> TO_SOT_Packages_SMD:SOT-223-3Lead_TabPin2
Connections:
- net +5V: now also D502.2 (A)
- net GND: now also R501.2
- new net: D502.1 (K), R501.1
Changed lines of the file:
@@
 F 0 "C501" H 5125 4350 50  0000 L CNN
 F 1 "4u7" H 5125 4150 50  0000 L CNN
-F 2 "Capacitors_SMD:CP_Elec_4x5.7" H 5138 4100 50  0001 C CNN
+F 2 "Capacitors_THT:CP_Radial_D6.3mm_P2.50mm" H 5138 4100 50  0001 C CNN
 F 3 "" H 5100 4250 50  0001 C CNN
 	1    5100 4250
@@
 F 0 "U501" H 5650 4125 50  0000 C CNN
 F 1 "AZ1117-5.0" H 5800 4125 50  0000 L CNN
-F 2 "TO_SOT_Packages_SMD:TO-263-3Lead" H 5800 4250 50  0001 C CIN
+F 2 "TO_SOT_Packages_SMD:SOT-223-3Lead_TabPin2" H 5800 4250 50  0001 C CIN
 F 3 "" H 5800 4000 50  0001 C CNN
 	1    5800 4000
@@
 F 0 "C504" H 6525 4350 50  0000 L CNN
 F 1 "47u" H 6525 4150 50  0000 L CNN
-F 2 "Capacitors_SMD:CP_Elec_4x5.7" H 6538 4100 50  0001 C CNN
+F 2 "Capacitors_THT:CP_Radial_D6.3mm_P2.50mm" H 6538 4100 50  0001 C CNN
 F 3 "" H 6500 4250 50  0001 C CNN
 	1    6500 4250
@@
 F 0 "C502" H 5425 4350 50  0000 L CNN
 F 1 "100n" H 5425 4150 50  0000 L CNN
-F 2 "Capacitors_SMD:C_1206" H 5438 4100 50  0001 C CNN
+F 2 "Capacitors_SMD:C_0805" H 5438 4100 50  0001 C CNN
 F 3 "" H 5400 4250 50  0001 C CNN
 	1    5400 4250
@@
 F 0 "C503" H 6225 4350 50  0000 L CNN
 F 1 "100n" H 6225 4150 50  0000 L CNN
-F 2 "Capacitors_SMD:C_1206" H 6238 4100 50  0001 C CNN
+F 2 "Capacitors_SMD:C_0805" H 6238 4100 50  0001 C CNN
 F 3 "" H 6200 4250 50  0001 C CNN
 	1    6200 4250
@@
 Wire Wire Line
 	5650 3700 5400 3700
+$Comp
+L LED D502
+U 1 1 59E32AE2
+P 7100 4050
+F 0 "D502" H 7100 4150 50  0000 C CNN
+F 1 "LED2" H 7100 3950 50  0000 C CNN
+F 2 "LEDs:LED_0805" H 7100 4050 50  0001 C CNN
+F 3 "" H 7100 4050 50  0001 C CNN
+	1    7100 4050
+	0    -1   -1   0
+$EndComp
+$Comp
+L R R501
+U 1 1 59E32AE9
+P 7100 4450
+F 0 "R501" V 7180 4450 50  0000 C CNN
+F 1 "430" V 7100 4450 50  0000 C CNN
+F 2 "Resistors_SMD:R_0805" V 7030 4450 50  0001 C CNN
+F 3 "" H 7100 4450 50  0001 C CNN
+	1    7100 4450
+	1    0    0    -1
+$EndComp
+$Comp
+L +5V #PWR057
+U 1 1 59E32AF0
+P 7100 3800
+F 0 "#PWR057" H 7100 3650 50  0001 C CNN
+F 1 "+5V" H 7100 3940 50  0000 C CNN
+F 2 "" H 7100 3800 50  0001 C CNN
+F 3 "" H 7100 3800 50  0001 C CNN
+	1    7100 3800
+	1    0    0    -1
+$EndComp
+Wire Wire Line
+	7100 3800 7100 3900
+Wire Wire Line
+	7100 4200 7100 4300
+$Comp
+L GND #PWR058
+U 1 1 59E32B42
+P 7100 4700
+F 0 "#PWR058" H 7100 4450 50  0001 C CNN
+F 1 "GND" H 7100 4550 50  0000 C CNN
+F 2 "" H 7100 4700 50  0001 C CNN
+F 3 "" H 7100 4700 50  0001 C CNN
+	1    7100 4700
+	1    0    0    -1
+$EndComp
+Wire Wire Line
+	7100 4700 7100 4600
 $EndSCHEMATC

Commit message: Kleine Veränderungen
Parts:
- C501: footprint Capacitors_THT:CP_Radial_D6.3mm_P2.50mm -> Capacitors_THT:CP_Radial_D5.0mm_P2.00mm
- D501: footprint Diodes_SMD:D_MiniMELF -> Diodes_SMD:D_SOD-123
Changed lines of the file:
@@
 F 0 "C501" H 5125 4350 50  0000 L CNN
 F 1 "4u7" H 5125 4150 50  0000 L CNN
-F 2 "Capacitors_THT:CP_Radial_D6.3mm_P2.50mm" H 5138 4100 50  0001 C CNN
+F 2 "Capacitors_THT:CP_Radial_D5.0mm_P2.00mm" H 5138 4100 50  0001 C CNN
 F 3 "" H 5100 4250 50  0001 C CNN
 	1    5100 4250
@@
 F 0 "D501" H 5800 3800 50  0000 C CNN
 F 1 "1N4148" H 5800 3600 50  0000 C CNN
-F 2 "Diodes_SMD:D_MiniMELF" H 5800 3700 50  0001 C CNN
+F 2 "Diodes_SMD:D_SOD-123" H 5800 3700 50  0001 C CNN
 F 3 "" H 5800 3700 50  0001 C CNN
 	1    5800 3700
