File: KiCad/button_mux.sch (KiCad schematic (older format))
At the start: 12 parts, among them J301 Button, U203 74LS00, U204 74LS126

Commit message: Applied changes for final design, placed test points.
Parts:
- C301: symbol C -> ledbox-rescue:C
- J301: symbol Conn_01x02 -> ledbox-rescue:Conn_01x02
- JP301: symbol Jumper_NO_Small -> ledbox-rescue:Jumper_NO_Small
- JP302: symbol Jumper_NC_Small -> ledbox-rescue:Jumper_NC_Small
- R301, R302: symbol R -> ledbox-rescue:R
- TP301, TP302, TP303, TP304: footprint Test:TEST_10 -> TestPoint:TestPoint_Pad_D1.0mm; symbol Test_Point -> ledbox-rescue:Test_Point
- U203: symbol 74LS00 -> ledbox-rescue:74LS00
- U204: symbol 74LS126 -> ledbox-rescue:74LS126
Connections:
- net BTN_DATA_IN: now also U204.9; no longer U204.2
- net BTN_LOAD: now also U203.12, U203.13, U204.13; no longer U203.10, U203.9, U204.4
- net BTN_OUT: now also U204.11, U204.8; no longer U204.3, U204.6
- net at JP301.2, JP302.1, R302.1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: now also U204.12; no longer U204.5
- new net: TP303.1, U203.11, U204.10
