File: KiCad/logic.sch (KiCad schematic (older format))
At the start: 27 parts, among them U201 74LS175, U202 74LS175, U203 74LS00, U204 74LS126

Commit message: Applied changes for final design, placed test points.
Parts:
- C201, C202, C203, C204: symbol C -> ledbox-rescue:C
- D201, D202: symbol LED -> ledbox-rescue:LED
- JP201, JP202, JP203, JP204: symbol Jumper_NC_Small -> ledbox-rescue:Jumper_NC_Small
- R201, R202: symbol R -> ledbox-rescue:R
- TP201, TP202, TP203, TP204, TP205, TP206, TP207, TP208, TP209, TP210, TP211: footprint Test:TEST_10 -> TestPoint:TestPoint_Pad_D1.0mm; symbol Test_Point -> ledbox-rescue:Test_Point
- U201, U202: symbol 74LS175 -> ledbox-rescue:74LS175
- U203: symbol 74LS00 -> ledbox-rescue:74LS00
- U204: symbol 74LS126 -> ledbox-rescue:74LS126
Connections:
- wire segments 84 -> 105
