File: KiCad/Interface.sch (KiCad schematic (older format))
At the start: 22 parts, among them J501 IR LED, Q501 NTR4003N, U501 WS2812B, U502 WS2812B, U503 WS2812B

Commit message: Applied changes for final design, placed test points.
Parts:
- removed Q501: NTR4003N, TO_SOT_Packages_SMD:SOT-23, symbol Q_NMOS_GSD
- added Q501: Q_PMOS_GSD, Package_TO_SOT_SMD:SOT-23, symbol Device:Q_PMOS_GSD
- C501, C502, C503, C504: symbol C -> ledbox-rescue:C
- J501: symbol Conn_01x03 -> ledbox-rescue:Conn_01x03
- JP501, JP502, JP503: symbol Jumper_NO_Small -> ledbox-rescue:Jumper_NO_Small
- R501, R502, R503, R504, R505: symbol R -> ledbox-rescue:R
- TP501, TP502, TP503, TP504, TP505: footprint Test:TEST_10 -> TestPoint:TestPoint_Pad_D1.0mm; symbol Test_Point -> ledbox-rescue:Test_Point
- U501, U502, U503: symbol WS2812B -> ledbox-rescue:WS2812B
Connections:
- wire segments 41 -> 53
Other:
- moved on the sheet: JP501, JP502, JP503, R501, R502, R503, R504, R505, TP503, TP504

Commit message: assigned transistor model
Parts:
- Q501: value Q_PMOS_GSD -> AO3415A
Changed lines of the file:
@@
 P 2650 1750
 F 0 "Q501" H 2856 1704 50  0000 L CNN
-F 1 "Q_PMOS_GSD" H 2856 1795 50  0000 L CNN
+F 1 "AO3415A" H 2856 1795 50  0000 L CNN
 F 2 "Package_TO_SOT_SMD:SOT-23" H 2850 1850 50  0001 C CNN
 F 3 "~" H 2650 1750 50  0001 C CNN

Commit message: paralleled RGB leds
Connections:
- wire segments 53 -> 59
Changed lines of the file:
@@
 	4800 4500 4800 4400
-Wire Wire Line
-	4700 5300 4800 5300
-Wire Wire Line
-	3200 5300 3300 5300
 Wire Wire Line
 	4200 4800 4200 4700
@@
 Wire Wire Line
 	3300 5200 3300 5300
-Connection ~ 3300 5300
 Wire Wire Line
 	4800 5200 4800 5300
-Connection ~ 4800 5300
 $Comp
 L ledbox-rescue:Jumper_NO_Small JP501
@@
 	7100 1300 7100 1500
 Wire Wire Line
-	1800 5300 2200 5300
-Wire Wire Line
-	3300 5300 3700 5300
-Wire Wire Line
-	4800 5300 5200 5300
+	1800 5300 2100 5300
 Wire Wire Line
 	2750 2850 3150 2850
@@
 Wire Wire Line
 	2350 1350 2350 1250
+Wire Wire Line
+	4700 5300 4800 5300
+Wire Wire Line
+	3200 5300 3300 5300
+Wire Wire Line
+	2100 5300 2100 6300
+Wire Wire Line
+	2100 6300 3600 6300
+Wire Wire Line
+	5100 6300 5100 5300
+Wire Wire Line
+	5100 5300 5200 5300
+Connection ~ 2100 5300
+Wire Wire Line
+	2100 5300 2200 5300
+Wire Wire Line
+	3700 5300 3600 5300
+Wire Wire Line
+	3600 5300 3600 6300
+Connection ~ 3600 6300
+Wire Wire Line
+	3600 6300 5100 6300
 $EndSCHEMATC
