File: KiCad/ledbox.kicad_pcb (KiCad board)
At the start: 2 copper layers, 80 x 50 mm, 88 parts, among them J101 Add Input, J102 5V, J103 To Master, J104 Add Output, J105 To Slave, J301 Button, J401 Button, J501 IR LED, Q501 AO3415A, U201 74LS175, U202 74LS175, U203 74LS00, U204 74LS126, U501 WS2812B, U502 WS2812B, U503 WS2812B

Commit message: Created final gerber files
Other:
- board text added: "5V"
- board text added: "BTN1"
- board text added: "BTN2"
- board text added: "F. Geissler RoboSAX LED Box V.4.2 “Shift Register”"
- board text added: "IN"
- board text added: "IR"
- board text added: "OUT"
- board text added: "To Master"
- board text added: "To Slave"
- board text removed: "F. Geissler RoboSAX LED Box V.4 “Shift Register”"
