File: KiCad/ledbox.kicad_pcb (KiCad board)
At the start: 2 copper layers, 80 x 50 mm, 88 parts, among them J101 Add Input, J102 5V, J103 To Master, J104 Add Output, J105 To Slave, J301 Button, J401 Button, J501 IR LED, Q501 AO3415A, U201 74LS175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

Commit message: turned data connectors to match cable layout
Parts:
- moved J103 10.5 mm to (117.5, 117.5), turned to 270 degrees
- moved J105 10.5 mm to (117.5, 130.8), turned to 270 degrees
Connections:
- J103 pad 1: GND -> /LED_DATA_IN
- J103 pad 10: /LED_DATA_IN -> GND
- J103 pad 2: /CLK -> /LED_LOAD
- J103 pad 3: GND -> /BTN_DATA_OUT
- J103 pad 4: /RGB_IN -> /BTN_LOAD
- J103 pad 5: GND -> /IR_CLK
- J103 pad 6: /IR_CLK -> GND
- J103 pad 7: /BTN_LOAD -> /RGB_IN
- J103 pad 8: /BTN_DATA_OUT -> GND
- J103 pad 9: /LED_LOAD -> /CLK
- J105 pad 1: GND -> /LED_DATA_OUT
- J105 pad 10: /LED_DATA_OUT -> GND
- J105 pad 2: /CLK -> /LED_LOAD
- J105 pad 3: GND -> /BTN_DATA_IN
- J105 pad 4: /RGB_OUT -> /BTN_LOAD
- J105 pad 5: GND -> /IR_CLK
- J105 pad 6: /IR_CLK -> GND
- J105 pad 7: /BTN_LOAD -> /RGB_OUT
- J105 pad 8: /BTN_DATA_IN -> GND
- J105 pad 9: /LED_LOAD -> /CLK
